Commit message: fix: tweaked sim lidar params

File: esda_sim/description/lidar.xacro (robot description, xacro)
@@ -21,5 +21,5 @@
         <parent link="base_link"/>
         <child link="velodyne"/>
-        <origin xyz="1 0 0.5" rpy="0 0 0"/>
+        <origin xyz="0.7 0 0.5" rpy="0 0 0"/>
     </joint>
     <gazebo reference="velodyne">
@@ -27,5 +27,5 @@
         <sensor name="laser" type="ray">
             <pose> 0 0 0 0 0 0 </pose>
-            <visualize>true</visualize>
+            <visualize>false</visualize>
             <update_rate>10</update_rate>
             <ray>
@@ -37,12 +37,12 @@
                     </horizontal>
                     <vertical>
-                        <samples>20</samples>
-                        <min_angle>-0.3</min_angle>
-                        <max_angle>0.3</max_angle>
+                        <samples>10</samples>
+                        <min_angle>-0.2</min_angle>
+                        <max_angle>0</max_angle>
                     </vertical>
                 </scan>
                 <range>
                     <min>0.3</min>
-                    <max>12</max>
+                    <max>4.5</max>
                 </range>
             </ray>
