Commit message: steering modelled with 4 front wheels, 1 left right to turn, 1 left right to spin

File: esda_sim/description/ackermann_control.xacro (robot description, xacro)
@@ -16,6 +16,6 @@
                axle rotation
           -->
-          <front_left_joint>left_steering_wheel_axle_joint</front_left_joint>
-          <front_right_joint>right_steering_wheel_axle_joint</front_right_joint>
+          <front_left_joint>left_wheel_axle_joint</front_left_joint>
+          <front_right_joint>right_wheel_axle_joint</front_right_joint>
           <!-- Arbitrary steering wheel to fulfil the API -->
           <steering_wheel_joint>steering_wheel_joint</steering_wheel_joint>

File: esda_sim/description/esda.urdf.xacro (robot description, xacro)
@@ -5,7 +5,8 @@
     <xacro:include filename="esda_core.xacro"/>
     <xacro:include filename="wheels.xacro"/>
-    <xacro:include filename="ackermann_control.xacro"/>
     <xacro:include filename="lidar.xacro"/>
     <xacro:include filename="piksi.xacro"/>
     <!--<xacro:include filename="camera.xacro"/>-->
+    <!--<xacro:include filename="ackermann_control.xacro"/>-->
+    <xacro:include filename="diff_control.xacro"/>
 </robot>

File: esda_sim/description/lidar.xacro (robot description, xacro)
@@ -23,5 +23,5 @@
         <parent link="base_link"/>
         <child link="velodyne"/>
-        <origin xyz="0.7 0 0.5" rpy="0 0 0"/>
+        <origin xyz="0 0 0.5" rpy="0 0 0"/>
     </joint>
     <gazebo reference="velodyne">

File: esda_sim/description/steering_wheels.xacro (robot description, xacro)
@@ -7,5 +7,5 @@
     <xacro:property name="steer_wheel_y_off" value="0.52297"/>
     <xacro:property name="steer_wheel_z_off" value="0.208"/>
-    <!-- Define the wheels themselves -->
+    <!-- Define the wheels that turn -->
     <link name="right_steering_wheel">
         <visual>
@@ -42,4 +42,39 @@
         </xacro:inertial_cylinder>
     </link>
+    <!-- Define the wheels that spin -->
+    <link name="right_axle_wheel">
+        <visual>
+            <geometry>
+                <cylinder radius="${wheel_rad}" length="${wheel_len}"/>
+            </geometry>
+            <material name="light_grey"/>
+        </visual>
+        <collision>
+            <geometry>
+                <cylinder radius="${wheel_rad}" length="${wheel_len}"/>
+            </geometry>
+            <material name="light_grey"/>
+        </collision>
+        <xacro:inertial_cylinder mass="${wheel_mass}" length="${wheel_len}" radius="${wheel_rad}">
+            <origin xyz="0 0 0" rpy="0 0 0"/>
+        </xacro:inertial_cylinder>
+    </link>
+    <link name="left_axle_wheel">
+        <visual>
+            <geometry>
+                <cylinder radius="${wheel_rad}" length="${wheel_len}"/>
+            </geometry>
+            <material name="light_grey"/>
+        </visual>
+        <collision>
+            <geometry>
+                <cylinder radius="${wheel_rad}" length="${wheel_len}"/>
+            </geometry>
+            <material name="light_grey"/>
+        </collision>
+        <xacro:inertial_cylinder mass="${wheel_mass}" length="${wheel_len}" radius="${wheel_rad}">
+            <origin xyz="0 0 0" rpy="0 0 0"/>
+        </xacro:inertial_cylinder>
+    </link>
     <!-- Note that in the following joint definitions, when defining the wheels
          axis of rotation, it refers to the wheel links axis, not base_link as
@@ -48,28 +83,30 @@
     -->
     <!-- Define the wheels rotation around the x axis so they can roll forward -->
-    <joint name="right_steering_wheel_axle_joint" type="continuous">
+    <joint name="right_wheel_axle_joint" type="continuous">
         <parent link="base_link"/>
-        <child link="right_steering_wheel"/>
+        <child link="right_axle_wheel"/>
         <origin xyz="${steer_wheel_x_off} -${steer_wheel_y_off} -${steer_wheel_z_off}" rpy="${pi/2} 0 0 "/>
         <axis xyz="0 0 1"/>
     </joint>
-    <joint name="left_steering_wheel_axle_joint" type="continuous">
+    <joint name="left_wheel_axle_joint" type="continuous">
         <parent link="base_link"/>
-        <child link="left_steering_wheel"/>
+        <child link="left_axle_wheel"/>
         <origin xyz="${steer_wheel_x_off} ${steer_wheel_y_off} -${steer_wheel_z_off}" rpy="-${pi/2} 0 0 "/>
         <axis xyz="0 0 -1"/>
     </joint>
     <!-- Define the wheels rotation around the z-axis so they can turn sideways -->
-    <joint name="right_steering_wheel_joint" type="continuous">
+    <joint name="right_steering_wheel_joint" type="revolute">
         <parent link="base_link"/>
         <child link="right_steering_wheel"/>
         <origin xyz="${steer_wheel_x_off} -${steer_wheel_y_off} -${steer_wheel_z_off}" rpy="${pi/2} 0 0 "/>
-        <axis xyz="0 1 0"/>
+        <axis xyz="0 -1 0"/>
+        <limit lower="-${6/10}" upper="${6/10}" effort="1" velocity="1"/>
     </joint>
-    <joint name="left_steering_wheel_joint" type="continuous">
+    <joint name="left_steering_wheel_joint" type="revolute">
         <parent link="base_link"/>
         <child link="left_steering_wheel"/>
         <origin xyz="${steer_wheel_x_off} ${steer_wheel_y_off} -${steer_wheel_z_off}" rpy="-${pi/2} 0 0 "/>
         <axis xyz="0 1 0"/>
+        <limit lower="-${6/10}" upper="${6/10}" effort="1" velocity="1"/>
     </joint>
     <!-- Define an arbitrary steering wheel as it's required for the AckermannControl plugin to work -->
@@ -94,5 +131,5 @@
         <parent link="base_link"/>
         <child link="steering_wheel"/>
-        <origin xyz="1 0 2" rpy="${pi/2} 0 ${pi/2}"/>
+        <origin xyz="0.5 0 0.5" rpy="${pi/2} 0 ${pi/2}"/>
         <axis xyz="0 0 1"/>
     </joint>
