Commit message: feat: added base footprint to urdf

File: esda_sim/description/esda_core.xacro (robot description, xacro)
@@ -22,6 +22,14 @@
          the datum point/point of reference and point that
          everything ultimately connects to
+         base_footprint is a child but has the same position
+         needed for SLAM toolbox
     -->
     <link name="base_link"></link>
+    <link name="base_footprint"></link>
+    <joint name="base_footprint_joint" type="fixed">
+        <parent link="base_link"/>
+        <child link="base_foot_print"/>
+        <origin xyz="0 0 0"/>
+    </joint>
     <!-- BODY LINKS
          these define the body of the ESDA which is simplified

Commit message: fix: updated esda sim body

File: esda_sim/description/esda_core.xacro (robot description, xacro)
@@ -38,18 +38,22 @@
     -->
     <!-- DRIVE BOX LINK -->
+    <xacro:property name="drive_box_x" value="0.5725"/>
+    <xacro:property name="drive_box_y" value="0.575"/>
+    <xacro:property name="drive_box_z" value="0.276"/>
+    <xacro:property name="drive_box_m" value="5"/>
     <link name="drive_box">
         <visual>
             <geometry>
-                <box size="0.505 0.57 0.275" />
-            </geometry>
-            <material name="white"/>
-        </visual>
-        <collision>
-            <geometry>
-                <box size="0.505 0.57 0.275" />
-            </geometry>
-            <material name="white"/>
-        </collision>
-        <xacro:inertial_box mass="5" x="0.505" y="0.57" z="0.275">
+                <box size="${drive_box_x} ${drive_box_y} ${drive_box_z}" />
+            </geometry>
+            <material name="white"/>
+        </visual>
+        <collision>
+            <geometry>
+                <box size="${drive_box_x} ${drive_box_y} ${drive_box_z}" />
+            </geometry>
+            <material name="white"/>
+        </collision>
+        <xacro:inertial_box mass="${drive_box_m}" x="${drive_box_x}" y="${drive_box_y}" z="${drive_box_z}">
             <origin xyz="0 0 0" rpy="0 0 0"/>
         </xacro:inertial_box>
@@ -58,51 +62,32 @@
         <parent link="base_link"/>
         <child link="drive_box"/>
-        <origin xyz="-0.2525 0 0"/>
-    </joint>
-    <!-- MIDDLE BOX LINK -->
-    <link name="middle_box">
-        <visual>
-            <geometry>
-                <box size="0.81 0.57 0.275" />
-            </geometry>
-            <material name="light_grey"/>
-        </visual>
-        <collision>
-            <geometry>
-                <box size="0.81 0.57 0.275" />
-            </geometry>
-            <material name="light_grey"/>
-        </collision>
-        <xacro:inertial_box mass="5" x="0.81" y="0.57" z="0.275">
+        <origin xyz="-0.28625 0 0"/>
+    </joint>
+    <!-- STEERING BOX LINK -->
+    <xacro:property name="steer_box_x" value="0.378"/>
+    <xacro:property name="steer_box_y" value="0.575"/>
+    <xacro:property name="steer_box_z" value="0.146"/>
+    <xacro:property name="steer_box_m" value="5"/>
+    <link name="steering_box">
+        <visual>
+            <geometry>
+                <box size="${steer_box_x} ${steer_box_y} ${steer_box_z}" />
+            </geometry>
+            <material name="white"/>
+        </visual>
+        <collision>
+            <geometry>
+                <box size="${steer_box_x} ${steer_box_y} ${steer_box_z}" />
+            </geometry>
+            <material name="white"/>
+        </collision>
+        <xacro:inertial_box mass="${steer_box_m}" x="${steer_box_x}" y="${steer_box_y}" z="${steer_box_z}">
             <origin xyz="0 0 0" rpy="0 0 0"/>
         </xacro:inertial_box>
     </link>
-    <joint name="middle_box_joint" type="fixed">
-        <parent link="base_link"/>
-        <child link="middle_box"/>
-        <origin xyz="0.405 0 0"/>
-    </joint>
-    <!-- STEERING BOX LINK -->
-    <link name="steering_box">
-        <visual>
-            <geometry>
-                <box size="0.505 0.57 0.275" />
-            </geometry>
-            <material name="white"/>
-        </visual>
-        <collision>
-            <geometry>
-                <box size="0.505 0.57 0.275" />
-            </geometry>
-            <material name="white"/>
-        </collision>
-        <xacro:inertial_box mass="5" x="0.505" y="0.57" z="0.275">
-            <origin xyz="0 0 0" rpy="0 0 0"/>
-        </xacro:inertial_box>
-    </link>
     <joint name="steering_box_joint" type="fixed">
         <parent link="base_link"/>
         <child link="steering_box"/>
-        <origin xyz="1.0625 0 0"/>
+        <origin xyz="0.189 0 -0.065"/>
     </joint>
     <!-- WHEEL LINKS

Commit message: fix: new body and wheel geom done

File: esda_sim/description/esda_core.xacro (robot description, xacro)
@@ -62,5 +62,5 @@
         <parent link="base_link"/>
         <child link="drive_box"/>
-        <origin xyz="-0.28625 0 0"/>
+        <origin xyz="-${drive_box_x/2} 0 0"/>
     </joint>
     <!-- STEERING BOX LINK -->
@@ -89,5 +89,5 @@
         <parent link="base_link"/>
         <child link="steering_box"/>
-        <origin xyz="0.189 0 -0.065"/>
+        <origin xyz="${steer_box_x/2} 0 -${drive_box_z/2-steer_box_z/2}"/> <!-- -0.065 -->
     </joint>
     <!-- WHEEL LINKS
@@ -98,5 +98,32 @@
     <xacro:property name="wheel_rad" value="0.1325"/>
     <xacro:property name="wheel_len" value="0.07"/>
-    <!-- LEFT DRIVE WHEEL -->
+    <xacro:property name="wheel_mass" value="2"/>
+    <!-- DRIVE WHEELS -->
+    <xacro:property name="drive_wheel_x_off" value="0.38724"/>
+    <xacro:property name="drive_wheel_y_off" value="0.48166"/>
+    <xacro:property name="drive_wheel_z_off" value="0.22"/>
+    <link name="right_drive_wheel">
+        <visual>
+            <geometry>
+                <cylinder radius="${wheel_rad}" length="${wheel_len}"/>
+            </geometry>
+            <material name="black"/>
+        </visual>
+        <collision>
+            <geometry>
+                <cylinder radius="${wheel_rad}" length="${wheel_len}"/>
+            </geometry>
+            <material name="black"/>
+        </collision>
+        <xacro:inertial_cylinder mass="${wheel_mass}" length="${wheel_len}" radius="${wheel_rad}">
+            <origin xyz="0 0 0" rpy="0 0 0"/>
+        </xacro:inertial_cylinder>
+    </link>
+    <joint name="right_drive_wheel_joint" type="continuous">
+        <parent link="base_link"/>
+        <child link="left_drive_wheel"/>
+        <origin xyz="-${drive_wheel_x_off} -${drive_wheel_y_off} -${drive_wheel_z_off}" rpy="${pi/2} 0 0 "/>
+        <axis xyz="0 0 1"/>
+    </joint>
     <link name="left_drive_wheel">
         <visual>
@@ -112,5 +139,5 @@
             <material name="black"/>
         </collision>
-        <xacro:inertial_cylinder mass="2" length="${wheel_len}" radius="${wheel_rad}">
+        <xacro:inertial_cylinder mass="${wheel_mass}" length="${wheel_len}" radius="${wheel_rad}">
             <origin xyz="0 0 0" rpy="0 0 0"/>
         </xacro:inertial_cylinder>
@@ -118,33 +145,35 @@
     <joint name="left_drive_wheel_joint" type="continuous">
         <parent link="base_link"/>
-        <child link="left_drive_wheel"/>
-        <origin xyz="-0.315 -0.479 -0.139" rpy="${pi/2} 0 0 "/>
+        <child link="right_drive_wheel"/>
+        <origin xyz="-${drive_wheel_x_off} ${drive_wheel_y_off} -${drive_wheel_z_off}" rpy="-${pi/2} 0 0 "/>
+        <axis xyz="0 0 -1"/>
+    </joint>
+   <!-- STEERING WHEELS -->
+    <xacro:property name="steer_wheel_x_off" value="0.235"/>
+    <xacro:property name="steer_wheel_y_off" value="0.52297"/>
+    <xacro:property name="steer_wheel_z_off" value="0.208"/>
+    <link name="right_steering_wheel">
+        <visual>
+            <geometry>
+                <cylinder radius="${wheel_rad}" length="${wheel_len}"/>
+            </geometry>
+            <material name="light_grey"/>
+        </visual>
+        <collision>
+            <geometry>
+                <cylinder radius="${wheel_rad}" length="${wheel_len}"/>
+            </geometry>
+            <material name="light_grey"/>
+        </collision>
+        <xacro:inertial_cylinder mass="${wheel_mass}" length="${wheel_len}" radius="${wheel_rad}">
+            <origin xyz="0 0 0" rpy="0 0 0"/>
+        </xacro:inertial_cylinder>
+    </link>
+    <joint name="right_steering_wheel_joint" type="continuous">
+        <parent link="base_link"/>
+        <child link="left_steering_wheel"/>
+        <origin xyz="${steer_wheel_x_off} -${steer_wheel_y_off} -${steer_wheel_z_off}" rpy="${pi/2} 0 0 "/>
         <axis xyz="0 0 1"/>
     </joint>
-    <!-- RIGHT DRIVE WHEEL -->
-    <link name="right_drive_wheel">
-        <visual>
-            <geometry>
-                <cylinder radius="${wheel_rad}" length="${wheel_len}"/>
-            </geometry>
-            <material name="black"/>
-        </visual>
-        <collision>
-            <geometry>
-                <cylinder radius="${wheel_rad}" length="${wheel_len}"/>
-            </geometry>
-            <material name="black"/>
-        </collision>
-        <xacro:inertial_cylinder mass="2" length="${wheel_len}" radius="${wheel_rad}">
-            <origin xyz="0 0 0" rpy="0 0 0"/>
-        </xacro:inertial_cylinder>
-    </link>
-    <joint name="right_drive_wheel_joint" type="continuous">
-        <parent link="base_link"/>
-        <child link="right_drive_wheel"/>
-        <origin xyz="-0.315 0.479 -0.139" rpy="-${pi/2} 0 0 "/>
-        <axis xyz="0 0 -1"/>
-    </joint>
-   <!-- LEFT STEERING WHEEL -->
     <link name="left_steering_wheel">
         <visual>
@@ -160,5 +189,5 @@
             <material name="light_grey"/>
         </collision>
-        <xacro:inertial_cylinder mass="2" length="${wheel_len}" radius="${wheel_rad}">
+        <xacro:inertial_cylinder mass="${wheel_mass}" length="${wheel_len}" radius="${wheel_rad}">
             <origin xyz="0 0 0" rpy="0 0 0"/>
         </xacro:inertial_cylinder>
@@ -166,30 +195,6 @@
     <joint name="left_steering_wheel_joint" type="continuous">
         <parent link="base_link"/>
-        <child link="left_steering_wheel"/>
-        <origin xyz="1.149 -0.51 -0.139" rpy="${pi/2} 0 0 "/>
-        <axis xyz="0 0 1"/>
-    </joint>
-    <!-- RIGHT STEERING WHEEL -->
-    <link name="right_steering_wheel">
-        <visual>
-            <geometry>
-                <cylinder radius="${wheel_rad}" length="${wheel_len}"/>
-            </geometry>
-            <material name="light_grey"/>
-        </visual>
-        <collision>
-            <geometry>
-                <cylinder radius="${wheel_rad}" length="${wheel_len}"/>
-            </geometry>
-            <material name="light_grey"/>
-        </collision>
-        <xacro:inertial_cylinder mass="2" length="${wheel_len}" radius="${wheel_rad}">
-            <origin xyz="0 0 0" rpy="0 0 0"/>
-        </xacro:inertial_cylinder>
-    </link>
-    <joint name="right_steering_wheel_joint" type="continuous">
-        <parent link="base_link"/>
         <child link="right_steering_wheel"/>
-        <origin xyz="1.149 0.51 -0.139" rpy="-${pi/2} 0 0 "/>
+        <origin xyz="${steer_wheel_x_off} ${steer_wheel_y_off} -${steer_wheel_z_off}" rpy="-${pi/2} 0 0 "/>
         <axis xyz="0 0 -1"/>
     </joint>

Commit message: feat added mid steer wheel to esda sim desc

File: esda_sim/description/esda_core.xacro (robot description, xacro)
@@ -172,5 +172,5 @@
     <joint name="right_steering_wheel_joint" type="continuous">
         <parent link="base_link"/>
-        <child link="left_steering_wheel"/>
+        <child link="right_steering_wheel"/>
         <origin xyz="${steer_wheel_x_off} -${steer_wheel_y_off} -${steer_wheel_z_off}" rpy="${pi/2} 0 0 "/>
         <axis xyz="0 0 1"/>
@@ -195,8 +195,31 @@
     <joint name="left_steering_wheel_joint" type="continuous">
         <parent link="base_link"/>
-        <child link="right_steering_wheel"/>
+        <child link="left_steering_wheel"/>
         <origin xyz="${steer_wheel_x_off} ${steer_wheel_y_off} -${steer_wheel_z_off}" rpy="-${pi/2} 0 0 "/>
         <axis xyz="0 0 -1"/>
     </joint>
+    <link name="mid_steering_wheel">
+        <visual>
+            <geometry>
+                <cylinder radius="${wheel_rad}" length="${wheel_len}"/>
+            </geometry>
+            <material name="light_grey"/>
+        </visual>
+        <collision>
+            <geometry>
+                <cylinder radius="${wheel_rad}" length="${wheel_len}"/>
+            </geometry>
+            <material name="light_grey"/>
+        </collision>
+        <xacro:inertial_cylinder mass="${wheel_mass}" length="${wheel_len}" radius="${wheel_rad}">
+            <origin xyz="0 0 0" rpy="0 0 0"/>
+        </xacro:inertial_cylinder>
+    </link>
+    <joint name="mid_steering_wheel_joint" type="continuous">
+        <parent link="base_link"/>
+        <child link="mid_steering_wheel"/>
+        <origin xyz="${steer_wheel_x_off} 0 -${steer_wheel_z_off}" rpy="-${pi/2} 0 0 "/>
+        <axis xyz="0 0 -1"/>
+    </joint>
     <!-- Adding colours to wheels for gazebo -->
     <gazebo reference="left_drive_wheel">

Commit message: feat: added wheel representing servo to model

File: esda_sim/description/esda_core.xacro (robot description, xacro)
@@ -222,4 +222,30 @@
         <axis xyz="0 0 -1"/>
     </joint>
+    <!-- SERVO -->
+    <xacro:property name="servo_x" value="0.05475"/>
+    <xacro:property name="servo_y" value="0.15"/>
+    <link name="servo">
+        <visual>
+            <geometry>
+                <cylinder radius="${wheel_rad}" length="${wheel_len}"/>
+            </geometry>
+            <material name="light_grey"/>
+        </visual>
+        <collision>
+            <geometry>
+                <cylinder radius="${wheel_rad}" length="${wheel_len}"/>
+            </geometry>
+            <material name="light_grey"/>
+        </collision>
+        <xacro:inertial_cylinder mass="${wheel_mass}" length="${wheel_len}" radius="${wheel_rad}">
+            <origin xyz="0 0 0" rpy="0 0 0"/>
+        </xacro:inertial_cylinder>
+    </link>
+    <joint name="servo_joint" type="continuous">
+        <parent link="base_link"/>
+        <child link="servo"/>
+        <origin xyz="${servo_x} ${servo_y} -${steer_wheel_z_off}" rpy="-${pi/2} 0 0 "/>
+        <axis xyz="0 0 -1"/>
+    </joint>
     <!-- Adding colours to wheels for gazebo -->
     <gazebo reference="left_drive_wheel">

Commit message: feat: added masses to componens in esda sim

File: esda_sim/description/esda_core.xacro (robot description, xacro)
@@ -23,5 +23,5 @@
     <xacro:property name="drive_box_y" value="0.575"/>
     <xacro:property name="drive_box_z" value="0.276"/>
-    <xacro:property name="drive_box_m" value="5"/>
+    <xacro:property name="drive_box_m" value="35"/>
     <link name="drive_box">
         <visual>
@@ -50,5 +50,5 @@
     <xacro:property name="steer_box_y" value="0.575"/>
     <xacro:property name="steer_box_z" value="0.146"/>
-    <xacro:property name="steer_box_m" value="5"/>
+    <xacro:property name="steer_box_m" value="29"/>
     <link name="steering_box">
         <visual>
