Commit message: is work

File: esda_sim/description/steering_wheels.xacro (robot description, xacro)
@@ -113,27 +113,3 @@
         <axis xyz="0 0 1"/>
     </joint>
-    <!-- Define an arbitrary steering wheel as it's required for the AckermannControl plugin to work -->
-    <link name="steering_wheel">
-        <visual>
-            <geometry>
-                <cylinder radius="0.1" length="0.1"/>
-            </geometry>
-            <material name="light_grey"/>
-        </visual>
-        <collision>
-            <geometry>
-                <cylinder radius="0.1" length="0.1"/>
-            </geometry>
-            <material name="black"/>
-        </collision>
-        <xacro:inertial_cylinder mass="0" length="0.1" radius="0.1">
-            <origin xyz="0 0 0" rpy="0 0 0"/>
-        </xacro:inertial_cylinder>
-    </link>
-    <joint name="steering_wheel_joint" type="continuous">
-        <parent link="base_link"/>
-        <child link="steering_wheel"/>
-        <origin xyz="0.1 0 0.1" rpy="0 0 0"/>
-        <axis xyz="0 0 1"/>
-    </joint>
 </robot>
