Commit message: fix: fixed esda launch errors

File: esda_sim/description/esda.urdf.xacro (robot description, xacro)
@@ -1,4 +1,13 @@
 <?xml version="1.0"?>
 <robot xmlns:xacro="http://www.ros.org/wiki/xacro" name="robot">
+    <material name="white">
+        <color rgba="1 1 1 1"/>
+    </material>
+    <material name="blue">
+        <color rgba="0.2 0.2 1 1"/>
+    </material>
+    <material name="orange">
+        <color rgba="1 0.3 0.1 1"/>
+    </material>
     <!-- ROOT LINK -->
     <!-- continue from here https://youtu.be/BcjHyhV0kIs?list=PLunhqkrRNRhYAffV8JDiFOatQXuU-NnxT&t=366 -->

Commit message: feat: added base of esda to urdf drive, steering and middle boxes

File: esda_sim/description/esda.urdf.xacro (robot description, xacro)
@@ -2,5 +2,8 @@
 <robot xmlns:xacro="http://www.ros.org/wiki/xacro" name="robot">
     <material name="white">
-        <color rgba="1 1 1 1"/>
+        <color rgba="1 1 1 0.3"/>
+    </material>
+    <material name="white2">
+        <color rgba="0.9 0.9 0.9 0.4"/>
     </material>
     <material name="blue">
@@ -13,3 +16,51 @@
     <!-- continue from here https://youtu.be/BcjHyhV0kIs?list=PLunhqkrRNRhYAffV8JDiFOatQXuU-NnxT&t=366 -->
     <link name="base_link"></link>
+    <!-- DRIVE BOX LINK -->
+    <link name="drive_box">
+        <visual>
+            <geometry>
+                <box size="0.505 0.57 0.275" />
+            </geometry>
+            <material name="white"/>
+        </visual>
+        <collision>
+        </collision>
+    </link>
+    <joint name="drive_box_joint" type="fixed">
+        <parent link="base_link"/>
+        <child link="drive_box"/>
+        <origin xyz="-0.2525 0 0"/>
+    </joint>
+    <!-- MIDDLE BOX -->
+    <link name="middle_box">
+        <visual>
+            <geometry>
+                <box size="0.81 0.57 0.275" />
+            </geometry>
+            <material name="white2"/>
+        </visual>
+        <collision>
+        </collision>
+    </link>
+    <joint name="middle_box_joint" type="fixed">
+        <parent link="base_link"/>
+        <child link="middle_box"/>
+        <origin xyz="0.405 0 0"/>
+    </joint>
+    <!-- STEERING BOX -->
+    <link name="steering_box">
+        <visual>
+            <geometry>
+                <box size="0.505 0.57 0.275" />
+            </geometry>
+            <material name="white"/>
+        </visual>
+        <collision>
+        </collision>
+    </link>
+    <joint name="steering_box_joint" type="fixed">
+        <parent link="base_link"/>
+        <child link="steering_box"/>
+        <origin xyz="1.0625 0 0"/>
+    </joint>
 </robot>

Commit message: feat: added drive wheels to robot desc

File: esda_sim/description/esda.urdf.xacro (robot description, xacro)
@@ -1,9 +1,13 @@
 <?xml version="1.0"?>
 <robot xmlns:xacro="http://www.ros.org/wiki/xacro" name="robot">
+    <!-- RANDOM COLOURS FOR DEBUG PURPOSES -->
     <material name="white">
         <color rgba="1 1 1 0.3"/>
     </material>
-    <material name="white2">
+    <material name="light_grey">
         <color rgba="0.9 0.9 0.9 0.4"/>
+    </material>
+    <material name="black">
+        <color rgba="0.2 0.2 0.2 0.4"/>
     </material>
     <material name="blue">
@@ -13,7 +17,13 @@
         <color rgba="1 0.3 0.1 1"/>
     </material>
-    <!-- ROOT LINK -->
-    <!-- continue from here https://youtu.be/BcjHyhV0kIs?list=PLunhqkrRNRhYAffV8JDiFOatQXuU-NnxT&t=366 -->
+    <!-- ROOT LINK
+         the datum point/point of reference and point that
+         everything ultimately connects to
+    -->
     <link name="base_link"></link>
+    <!-- BODY LINKS
+         these define the body of the ESDA which is simplified
+         as a series of boxes
+    -->
     <!-- DRIVE BOX LINK -->
     <link name="drive_box">
@@ -24,6 +34,4 @@
             <material name="white"/>
         </visual>
-        <collision>
-        </collision>
     </link>
     <joint name="drive_box_joint" type="fixed">
@@ -32,5 +40,5 @@
         <origin xyz="-0.2525 0 0"/>
     </joint>
-    <!-- MIDDLE BOX -->
+    <!-- MIDDLE BOX LINK -->
     <link name="middle_box">
         <visual>
@@ -38,8 +46,6 @@
                 <box size="0.81 0.57 0.275" />
             </geometry>
-            <material name="white2"/>
+            <material name="light_grey"/>
         </visual>
-        <collision>
-        </collision>
     </link>
     <joint name="middle_box_joint" type="fixed">
@@ -48,5 +54,5 @@
         <origin xyz="0.405 0 0"/>
     </joint>
-    <!-- STEERING BOX -->
+    <!-- STEERING BOX LINK -->
     <link name="steering_box">
         <visual>
@@ -56,6 +62,4 @@
             <material name="white"/>
         </visual>
-        <collision>
-        </collision>
     </link>
     <joint name="steering_box_joint" type="fixed">
@@ -64,3 +68,38 @@
         <origin xyz="1.0625 0 0"/>
     </joint>
+    <!-- WHEEL LINKS
+         these define the 4 wheels and their attachment to
+         the vehicle. Note due to complexity of CAD, wheels are
+         parallel and upright as they don't need accurate modelling
+    -->
+    <!-- DRIVE WHEELS -->
+    <link name="left_drive_wheel">
+        <visual>
+            <geometry>
+                <cylinder radius="0.1325" length="0.07"/>
+            </geometry>
+            <material name="light_grey"/>
+        </visual>
+    </link>
+    <joint name="left_drive_wheel_joint" type="continuous">
+        <parent link="base_link"/>
+        <child link="left_drive_wheel"/>
+        <origin xyz="-0.315 -0.479 -0.139" rpy="${pi/2} 0 0 "/>
+        <axis xyz="0 0 1"/>
+    </joint>
+    <link name="right_drive_wheel">
+        <visual>
+            <geometry>
+                <cylinder radius="0.1325" length="0.07"/>
+            </geometry>
+            <material name="light_grey"/>
+        </visual>
+    </link>
+    <joint name="right_drive_wheel_joint" type="continuous">
+        <parent link="base_link"/>
+        <child link="right_drive_wheel"/>
+        <origin xyz="-0.315 0.479 -0.139" rpy="-${pi/2} 0 0 "/>
+        <axis xyz="0 0 -1"/>
+    </joint>
+    <!-- STEERING WHEELS -->
 </robot>

Commit message: feat: added collision elements to components

File: esda_sim/description/esda.urdf.xacro (robot description, xacro)
@@ -34,4 +34,10 @@
             <material name="white"/>
         </visual>
+        <collision>
+            <geometry>
+                <box size="0.505 0.57 0.275" />
+            </geometry>
+            <material name="white"/>
+        </collision>
     </link>
     <joint name="drive_box_joint" type="fixed">
@@ -48,4 +54,10 @@
             <material name="light_grey"/>
         </visual>
+        <collision>
+            <geometry>
+                <box size="0.81 0.57 0.275" />
+            </geometry>
+            <material name="light_grey"/>
+        </collision>
     </link>
     <joint name="middle_box_joint" type="fixed">
@@ -62,4 +74,10 @@
             <material name="white"/>
         </visual>
+        <collision>
+            <geometry>
+                <box size="0.505 0.57 0.275" />
+            </geometry>
+            <material name="white"/>
+        </collision>
     </link>
     <joint name="steering_box_joint" type="fixed">
@@ -73,5 +91,5 @@
          parallel and upright as they don't need accurate modelling
     -->
-    <!-- DRIVE WHEELS -->
+    <!-- LEFT DRIVE WHEEL -->
     <link name="left_drive_wheel">
         <visual>
@@ -79,6 +97,12 @@
                 <cylinder radius="0.1325" length="0.07"/>
             </geometry>
-            <material name="light_grey"/>
+            <material name="black"/>
         </visual>
+        <collision>
+            <geometry>
+                <cylinder radius="0.1325" length="0.07"/>
+            </geometry>
+            <material name="black"/>
+        </collision>
     </link>
     <joint name="left_drive_wheel_joint" type="continuous">
@@ -88,4 +112,5 @@
         <axis xyz="0 0 1"/>
     </joint>
+    <!-- RIGHT DRIVE WHEEL -->
     <link name="right_drive_wheel">
         <visual>
@@ -93,6 +118,12 @@
                 <cylinder radius="0.1325" length="0.07"/>
             </geometry>
-            <material name="light_grey"/>
+            <material name="black"/>
         </visual>
+        <collision>
+            <geometry>
+                <cylinder radius="0.1325" length="0.07"/>
+            </geometry>
+            <material name="black"/>
+        </collision>
     </link>
     <joint name="right_drive_wheel_joint" type="continuous">
@@ -102,4 +133,45 @@
         <axis xyz="0 0 -1"/>
     </joint>
-    <!-- STEERING WHEELS -->
+   <!-- LEFT STEERING WHEEL -->
+    <link name="left_steering_wheel">
+        <visual>
+            <geometry>
+                <cylinder radius="0.1325" length="0.07"/>
+            </geometry>
+            <material name="light_grey"/>
+        </visual>
+        <collision>
+            <geometry>
+                <cylinder radius="0.1325" length="0.07"/>
+            </geometry>
+            <material name="light_grey"/>
+        </collision>
+    </link>
+    <joint name="left_steering_wheel_joint" type="continuous">
+        <parent link="base_link"/>
+        <child link="left_steering_wheel"/>
+        <origin xyz="1.149 -0.51 -0.139" rpy="${pi/2} 0 0 "/>
+        <axis xyz="0 0 1"/>
+    </joint>
+    <!-- RIGHT STEERING WHEEL -->
+    <link name="right_steering_wheel">
+        <visual>
+            <geometry>
+                <cylinder radius="0.1325" length="0.07"/>
+            </geometry>
+            <material name="light_grey"/>
+        </visual>
+        <collision>
+            <geometry>
+                <cylinder radius="0.1325" length="0.07"/>
+            </geometry>
+            <material name="light_grey"/>
+        </collision>
+    </link>
+    <joint name="right_steering_wheel_joint" type="continuous">
+        <parent link="base_link"/>
+        <child link="right_steering_wheel"/>
+        <origin xyz="1.149 0.51 -0.139" rpy="-${pi/2} 0 0 "/>
+        <axis xyz="0 0 -1"/>
+    </joint>
 </robot>

Commit message: fix: added inertial tags and now robot spawns in gazebo

File: esda_sim/description/esda.urdf.xacro (robot description, xacro)
@@ -1,4 +1,6 @@
 <?xml version="1.0"?>
 <robot xmlns:xacro="http://www.ros.org/wiki/xacro" name="robot">
+    <!-- IMPORTS -->
+    <xacro:include filename="inertial_macros.xacro"/>
     <!-- RANDOM COLOURS FOR DEBUG PURPOSES -->
     <material name="white">
@@ -40,4 +42,7 @@
             <material name="white"/>
         </collision>
+        <xacro:inertial_box mass="5" x="0.505" y="0.57" z="0.275">
+            <origin xyz="0 0 0" rpy="0 0 0"/>
+        </xacro:inertial_box>
     </link>
     <joint name="drive_box_joint" type="fixed">
@@ -60,4 +65,7 @@
             <material name="light_grey"/>
         </collision>
+        <xacro:inertial_box mass="5" x="0.81" y="0.57" z="0.275">
+            <origin xyz="0 0 0" rpy="0 0 0"/>
+        </xacro:inertial_box>
     </link>
     <joint name="middle_box_joint" type="fixed">
@@ -80,4 +88,7 @@
             <material name="white"/>
         </collision>
+        <xacro:inertial_box mass="5" x="0.505" y="0.57" z="0.275">
+            <origin xyz="0 0 0" rpy="0 0 0"/>
+        </xacro:inertial_box>
     </link>
     <joint name="steering_box_joint" type="fixed">
@@ -105,4 +116,7 @@
             <material name="black"/>
         </collision>
+        <xacro:inertial_cylinder mass="1" length="0.07" radius="0.1325">
+            <origin xyz="0 0 0" rpy="0 0 0"/>
+        </xacro:inertial_cylinder>
     </link>
     <joint name="left_drive_wheel_joint" type="continuous">
@@ -126,4 +140,7 @@
             <material name="black"/>
         </collision>
+        <xacro:inertial_cylinder mass="1" length="0.07" radius="0.1325">
+            <origin xyz="0 0 0" rpy="0 0 0"/>
+        </xacro:inertial_cylinder>
     </link>
     <joint name="right_drive_wheel_joint" type="continuous">
@@ -147,4 +164,7 @@
             <material name="light_grey"/>
         </collision>
+        <xacro:inertial_box mass="5" x="0.505" y="0.57" z="0.275">
+            <origin xyz="0 0 0" rpy="0 0 0"/>
+        </xacro:inertial_box>
     </link>
     <joint name="left_steering_wheel_joint" type="continuous">
@@ -168,4 +188,7 @@
             <material name="light_grey"/>
         </collision>
+        <xacro:inertial_box mass="5" x="0.505" y="0.57" z="0.275">
+            <origin xyz="0 0 0" rpy="0 0 0"/>
+        </xacro:inertial_box>
     </link>
     <joint name="right_steering_wheel_joint" type="continuous">

Commit message: feat: esda runs in gazebo with teleop twist kb using diff

File: esda_sim/description/esda.urdf.xacro (robot description, xacro)
@@ -1,200 +1,5 @@
 <?xml version="1.0"?>
 <robot xmlns:xacro="http://www.ros.org/wiki/xacro" name="robot">
-    <!-- IMPORTS -->
-    <xacro:include filename="inertial_macros.xacro"/>
-    <!-- RANDOM COLOURS FOR DEBUG PURPOSES -->
-    <material name="white">
-        <color rgba="1 1 1 0.3"/>
-    </material>
-    <material name="light_grey">
-        <color rgba="0.9 0.9 0.9 0.4"/>
-    </material>
-    <material name="black">
-        <color rgba="0.2 0.2 0.2 0.4"/>
-    </material>
-    <material name="blue">
-        <color rgba="0.2 0.2 1 1"/>
-    </material>
-    <material name="orange">
-        <color rgba="1 0.3 0.1 1"/>
-    </material>
-    <!-- ROOT LINK
-         the datum point/point of reference and point that
-         everything ultimately connects to
-    -->
-    <link name="base_link"></link>
-    <!-- BODY LINKS
-         these define the body of the ESDA which is simplified
-         as a series of boxes
-    -->
-    <!-- DRIVE BOX LINK -->
-    <link name="drive_box">
-        <visual>
-            <geometry>
-                <box size="0.505 0.57 0.275" />
-            </geometry>
-            <material name="white"/>
-        </visual>
-        <collision>
-            <geometry>
-                <box size="0.505 0.57 0.275" />
-            </geometry>
-            <material name="white"/>
-        </collision>
-        <xacro:inertial_box mass="5" x="0.505" y="0.57" z="0.275">
-            <origin xyz="0 0 0" rpy="0 0 0"/>
-        </xacro:inertial_box>
-    </link>
-    <joint name="drive_box_joint" type="fixed">
-        <parent link="base_link"/>
-        <child link="drive_box"/>
-        <origin xyz="-0.2525 0 0"/>
-    </joint>
-    <!-- MIDDLE BOX LINK -->
-    <link name="middle_box">
-        <visual>
-            <geometry>
-                <box size="0.81 0.57 0.275" />
-            </geometry>
-            <material name="light_grey"/>
-        </visual>
-        <collision>
-            <geometry>
-                <box size="0.81 0.57 0.275" />
-            </geometry>
-            <material name="light_grey"/>
-        </collision>
-        <xacro:inertial_box mass="5" x="0.81" y="0.57" z="0.275">
-            <origin xyz="0 0 0" rpy="0 0 0"/>
-        </xacro:inertial_box>
-    </link>
-    <joint name="middle_box_joint" type="fixed">
-        <parent link="base_link"/>
-        <child link="middle_box"/>
-        <origin xyz="0.405 0 0"/>
-    </joint>
-    <!-- STEERING BOX LINK -->
-    <link name="steering_box">
-        <visual>
-            <geometry>
-                <box size="0.505 0.57 0.275" />
-            </geometry>
-            <material name="white"/>
-        </visual>
-        <collision>
-            <geometry>
-                <box size="0.505 0.57 0.275" />
-            </geometry>
-            <material name="white"/>
-        </collision>
-        <xacro:inertial_box mass="5" x="0.505" y="0.57" z="0.275">
-            <origin xyz="0 0 0" rpy="0 0 0"/>
-        </xacro:inertial_box>
-    </link>
-    <joint name="steering_box_joint" type="fixed">
-        <parent link="base_link"/>
-        <child link="steering_box"/>
-        <origin xyz="1.0625 0 0"/>
-    </joint>
-    <!-- WHEEL LINKS
-         these define the 4 wheels and their attachment to
-         the vehicle. Note due to complexity of CAD, wheels are
-         parallel and upright as they don't need accurate modelling
-    -->
-    <!-- LEFT DRIVE WHEEL -->
-    <link name="left_drive_wheel">
-        <visual>
-            <geometry>
-                <cylinder radius="0.1325" length="0.07"/>
-            </geometry>
-            <material name="black"/>
-        </visual>
-        <collision>
-            <geometry>
-                <cylinder radius="0.1325" length="0.07"/>
-            </geometry>
-            <material name="black"/>
-        </collision>
-        <xacro:inertial_cylinder mass="1" length="0.07" radius="0.1325">
-            <origin xyz="0 0 0" rpy="0 0 0"/>
-        </xacro:inertial_cylinder>
-    </link>
-    <joint name="left_drive_wheel_joint" type="continuous">
-        <parent link="base_link"/>
-        <child link="left_drive_wheel"/>
-        <origin xyz="-0.315 -0.479 -0.139" rpy="${pi/2} 0 0 "/>
-        <axis xyz="0 0 1"/>
-    </joint>
-    <!-- RIGHT DRIVE WHEEL -->
-    <link name="right_drive_wheel">
-        <visual>
-            <geometry>
-                <cylinder radius="0.1325" length="0.07"/>
-            </geometry>
-            <material name="black"/>
-        </visual>
-        <collision>
-            <geometry>
-                <cylinder radius="0.1325" length="0.07"/>
-            </geometry>
-            <material name="black"/>
-        </collision>
-        <xacro:inertial_cylinder mass="1" length="0.07" radius="0.1325">
-            <origin xyz="0 0 0" rpy="0 0 0"/>
-        </xacro:inertial_cylinder>
-    </link>
-    <joint name="right_drive_wheel_joint" type="continuous">
-        <parent link="base_link"/>
-        <child link="right_drive_wheel"/>
-        <origin xyz="-0.315 0.479 -0.139" rpy="-${pi/2} 0 0 "/>
-        <axis xyz="0 0 -1"/>
-    </joint>
-   <!-- LEFT STEERING WHEEL -->
-    <link name="left_steering_wheel">
-        <visual>
-            <geometry>
-                <cylinder radius="0.1325" length="0.07"/>
-            </geometry>
-            <material name="light_grey"/>
-        </visual>
-        <collision>
-            <geometry>
-                <cylinder radius="0.1325" length="0.07"/>
-            </geometry>
-            <material name="light_grey"/>
-        </collision>
-        <xacro:inertial_box mass="5" x="0.505" y="0.57" z="0.275">
-            <origin xyz="0 0 0" rpy="0 0 0"/>
-        </xacro:inertial_box>
-    </link>
-    <joint name="left_steering_wheel_joint" type="continuous">
-        <parent link="base_link"/>
-        <child link="left_steering_wheel"/>
-        <origin xyz="1.149 -0.51 -0.139" rpy="${pi/2} 0 0 "/>
-        <axis xyz="0 0 1"/>
-    </joint>
-    <!-- RIGHT STEERING WHEEL -->
-    <link name="right_steering_wheel">
-        <visual>
-            <geometry>
-                <cylinder radius="0.1325" length="0.07"/>
-            </geometry>
-            <material name="light_grey"/>
-        </visual>
-        <collision>
-            <geometry>
-                <cylinder radius="0.1325" length="0.07"/>
-            </geometry>
-            <material name="light_grey"/>
-        </collision>
-        <xacro:inertial_box mass="5" x="0.505" y="0.57" z="0.275">
-            <origin xyz="0 0 0" rpy="0 0 0"/>
-        </xacro:inertial_box>
-    </link>
-    <joint name="right_steering_wheel_joint" type="continuous">
-        <parent link="base_link"/>
-        <child link="right_steering_wheel"/>
-        <origin xyz="1.149 0.51 -0.139" rpy="-${pi/2} 0 0 "/>
-        <axis xyz="0 0 -1"/>
-    </joint>
+    <xacro:include filename="esda_core.xacro"/>
+    <xacro:include filename="gazebo_control.xacro"/>
 </robot>

Commit message: fix/feat: urdf wheel inertials all cylindar, added lidar xacro

File: esda_sim/description/esda.urdf.xacro (robot description, xacro)
@@ -3,3 +3,4 @@
     <xacro:include filename="esda_core.xacro"/>
     <xacro:include filename="gazebo_control.xacro"/>
+    <xacro:include filename="lidar.xacro"/>
 </robot>

File: esda_sim/description/esda_core.xacro (robot description, xacro)
@@ -116,5 +116,5 @@
             <material name="black"/>
         </collision>
-        <xacro:inertial_cylinder mass="1" length="0.07" radius="0.1325">
+        <xacro:inertial_cylinder mass="2" length="0.07" radius="0.1325">
             <origin xyz="0 0 0" rpy="0 0 0"/>
         </xacro:inertial_cylinder>
@@ -140,5 +140,5 @@
             <material name="black"/>
         </collision>
-        <xacro:inertial_cylinder mass="1" length="0.07" radius="0.1325">
+        <xacro:inertial_cylinder mass="2" length="0.07" radius="0.1325">
             <origin xyz="0 0 0" rpy="0 0 0"/>
         </xacro:inertial_cylinder>
@@ -164,7 +164,7 @@
             <material name="light_grey"/>
         </collision>
-        <xacro:inertial_box mass="5" x="0.505" y="0.57" z="0.275">
-            <origin xyz="0 0 0" rpy="0 0 0"/>
-        </xacro:inertial_box>
+        <xacro:inertial_cylinder mass="2" length="0.07" radius="0.1325">
+            <origin xyz="0 0 0" rpy="0 0 0"/>
+        </xacro:inertial_cylinder>
     </link>
     <joint name="left_steering_wheel_joint" type="continuous">
@@ -188,7 +188,7 @@
             <material name="light_grey"/>
         </collision>
-        <xacro:inertial_box mass="5" x="0.505" y="0.57" z="0.275">
-            <origin xyz="0 0 0" rpy="0 0 0"/>
-        </xacro:inertial_box>
+        <xacro:inertial_cylinder mass="2" length="0.07" radius="0.1325">
+            <origin xyz="0 0 0" rpy="0 0 0"/>
+        </xacro:inertial_cylinder>
     </link>
     <joint name="right_steering_wheel_joint" type="continuous">

Commit message: fix: base_footprint joint in esda.urdf.xacro

File: esda_sim/description/esda.urdf.xacro (robot description, xacro)
@@ -4,4 +4,4 @@
     <xacro:include filename="gazebo_control.xacro"/>
     <xacro:include filename="lidar.xacro"/>
-    <xacro:include filename="camera.xacro"/>
+    <!--<xacro:include filename="camera.xacro"/>-->
 </robot>

File: esda_sim/description/esda_core.xacro (robot description, xacro)
@@ -22,12 +22,13 @@
          the datum point/point of reference and point that
          everything ultimately connects to
-         base_footprint is a child but has the same position
-         needed for SLAM toolbox
     -->
     <link name="base_link"></link>
+    <!-- base_footprint is a child but of base_link but
+         has the same position as its needed for SLAM toolbox
+    -->
     <link name="base_footprint"></link>
     <joint name="base_footprint_joint" type="fixed">
         <parent link="base_link"/>
-        <child link="base_foot_print"/>
+        <child link="base_footprint"/>
         <origin xyz="0 0 0"/>
     </joint>
