Commit message: feat: added placeholder box for piksi in sim

File: esda_sim/description/esda.urdf.xacro (robot description, xacro)
@@ -4,4 +4,5 @@
     <xacro:include filename="gazebo_control.xacro"/>
     <xacro:include filename="lidar.xacro"/>
+    <xacro:include filename="piksi.xacro"/>
     <!--<xacro:include filename="camera.xacro"/>-->
 </robot>

File: esda_sim/description/esda_core.xacro (robot description, xacro)
@@ -111,19 +111,21 @@
          parallel and upright as they don't need accurate modelling
     -->
+    <xacro:property name="wheel_rad" value="0.1325"/>
+    <xacro:property name="wheel_len" value="0.07"/>
     <!-- LEFT DRIVE WHEEL -->
     <link name="left_drive_wheel">
         <visual>
             <geometry>
-                <cylinder radius="0.1325" length="0.07"/>
-            </geometry>
-            <material name="black"/>
-        </visual>
-        <collision>
-            <geometry>
-                <cylinder radius="0.1325" length="0.07"/>
-            </geometry>
-            <material name="black"/>
-        </collision>
-        <xacro:inertial_cylinder mass="2" length="0.07" radius="0.1325">
+                <cylinder radius="${wheel_rad}" length="${wheel_len}"/>
+            </geometry>
+            <material name="black"/>
+        </visual>
+        <collision>
+            <geometry>
+                <cylinder radius="${wheel_rad}" length="${wheel_len}"/>
+            </geometry>
+            <material name="black"/>
+        </collision>
+        <xacro:inertial_cylinder mass="2" length="${wheel_len}" radius="${wheel_rad}">
             <origin xyz="0 0 0" rpy="0 0 0"/>
         </xacro:inertial_cylinder>
@@ -139,15 +141,15 @@
         <visual>
             <geometry>
-                <cylinder radius="0.1325" length="0.07"/>
-            </geometry>
-            <material name="black"/>
-        </visual>
-        <collision>
-            <geometry>
-                <cylinder radius="0.1325" length="0.07"/>
-            </geometry>
-            <material name="black"/>
-        </collision>
-        <xacro:inertial_cylinder mass="2" length="0.07" radius="0.1325">
+                <cylinder radius="${wheel_rad}" length="${wheel_len}"/>
+            </geometry>
+            <material name="black"/>
+        </visual>
+        <collision>
+            <geometry>
+                <cylinder radius="${wheel_rad}" length="${wheel_len}"/>
+            </geometry>
+            <material name="black"/>
+        </collision>
+        <xacro:inertial_cylinder mass="2" length="${wheel_len}" radius="${wheel_rad}">
             <origin xyz="0 0 0" rpy="0 0 0"/>
         </xacro:inertial_cylinder>
@@ -163,15 +165,15 @@
         <visual>
             <geometry>
-                <cylinder radius="0.1325" length="0.07"/>
-            </geometry>
-            <material name="light_grey"/>
-        </visual>
-        <collision>
-            <geometry>
-                <cylinder radius="0.1325" length="0.07"/>
-            </geometry>
-            <material name="light_grey"/>
-        </collision>
-        <xacro:inertial_cylinder mass="2" length="0.07" radius="0.1325">
+                <cylinder radius="${wheel_rad}" length="${wheel_len}"/>
+            </geometry>
+            <material name="light_grey"/>
+        </visual>
+        <collision>
+            <geometry>
+                <cylinder radius="${wheel_rad}" length="${wheel_len}"/>
+            </geometry>
+            <material name="light_grey"/>
+        </collision>
+        <xacro:inertial_cylinder mass="2" length="${wheel_len}" radius="${wheel_rad}">
             <origin xyz="0 0 0" rpy="0 0 0"/>
         </xacro:inertial_cylinder>
@@ -187,15 +189,15 @@
         <visual>
             <geometry>
-                <cylinder radius="0.1325" length="0.07"/>
-            </geometry>
-            <material name="light_grey"/>
-        </visual>
-        <collision>
-            <geometry>
-                <cylinder radius="0.1325" length="0.07"/>
-            </geometry>
-            <material name="light_grey"/>
-        </collision>
-        <xacro:inertial_cylinder mass="2" length="0.07" radius="0.1325">
+                <cylinder radius="${wheel_rad}" length="${wheel_len}"/>
+            </geometry>
+            <material name="light_grey"/>
+        </visual>
+        <collision>
+            <geometry>
+                <cylinder radius="${wheel_rad}" length="${wheel_len}"/>
+            </geometry>
+            <material name="light_grey"/>
+        </collision>
+        <xacro:inertial_cylinder mass="2" length="${wheel_len}" radius="${wheel_rad}">
             <origin xyz="0 0 0" rpy="0 0 0"/>
         </xacro:inertial_cylinder>

File: esda_sim/description/lidar.xacro (robot description, xacro)
@@ -1,8 +1,10 @@
 <?xml version="1.0"?>
 <robot xmlns:xacro="http://www.ros.org/wiki/xacro">
+    <xacro:property name="lidar_rad" value="0.0515"/>
+    <xacro:property name="lidar_len" value="0.072"/>
     <link name="velodyne">
         <visual>
             <geometry>
-                <cylinder radius="0.1" length="0.1"/>
+                <cylinder radius="${lidar_rad}" length="${lidar_len}"/>
             </geometry>
             <material name="orange"/>
@@ -10,9 +12,9 @@
         <collision>
             <geometry>
-                <cylinder radius="0.1325" length="0.07"/>
+                <cylinder radius="${lidar_rad}" length="${lidar_len}"/>
             </geometry>
             <material name="orange"/>
         </collision>
-        <xacro:inertial_cylinder mass="1" length="0.07" radius="0.1325">
+        <xacro:inertial_cylinder mass="1" radius="${lidar_rad}" length="${lidar_len}">
             <origin xyz="0 0 0" rpy="0 0 0"/>
         </xacro:inertial_cylinder>

Commit message: feat: ackerman control plugin integratio with esda urdf

File: esda_sim/description/esda.urdf.xacro (robot description, xacro)
@@ -1,6 +1,9 @@
 <?xml version="1.0"?>
 <robot xmlns:xacro="http://www.ros.org/wiki/xacro" name="robot">
+    <xacro:include filename="inertial_macros.xacro"/>
+    <xacro:include filename="materials.xacro"/>
     <xacro:include filename="esda_core.xacro"/>
-    <xacro:include filename="gazebo_control.xacro"/>
+    <xacro:include filename="wheels.xacro"/>
+    <xacro:include filename="ackermann_control.xacro"/>
     <xacro:include filename="lidar.xacro"/>
     <xacro:include filename="piksi.xacro"/>

File: esda_sim/description/esda_core.xacro (robot description, xacro)
@@ -1,22 +1,4 @@
 <?xml version="1.0"?>
 <robot xmlns:xacro="http://www.ros.org/wiki/xacro">
-    <!-- IMPORTS -->
-    <xacro:include filename="inertial_macros.xacro"/>
-    <!-- RANDOM COLOURS FOR DEBUG PURPOSES -->
-    <material name="white">
-        <color rgba="1 1 1 0.3"/>
-    </material>
-    <material name="light_grey">
-        <color rgba="0.9 0.9 0.9 0.4"/>
-    </material>
-    <material name="black">
-        <color rgba="0.2 0.2 0.2 0.4"/>
-    </material>
-    <material name="blue">
-        <color rgba="0.2 0.2 1 1"/>
-    </material>
-    <material name="orange">
-        <color rgba="1 0.3 0.1 1"/>
-    </material>
     <!-- ROOT LINK
          the datum point/point of reference and point that
@@ -91,173 +73,3 @@
         <origin xyz="${steer_box_x/2} 0 -${drive_box_z/2-steer_box_z/2}"/> <!-- -0.065 -->
     </joint>
-    <!-- WHEEL LINKS
-         these define the 4 wheels and their attachment to
-         the vehicle. Note due to complexity of CAD, wheels are
-         parallel and upright as they don't need accurate modelling
-    -->
-    <xacro:property name="wheel_rad" value="0.1325"/>
-    <xacro:property name="wheel_len" value="0.07"/>
-    <xacro:property name="wheel_mass" value="2"/>
-    <!-- DRIVE WHEELS -->
-    <xacro:property name="drive_wheel_x_off" value="0.38724"/>
-    <xacro:property name="drive_wheel_y_off" value="0.48166"/>
-    <xacro:property name="drive_wheel_z_off" value="0.22"/>
-    <link name="right_drive_wheel">
-        <visual>
-            <geometry>
-                <cylinder radius="${wheel_rad}" length="${wheel_len}"/>
-            </geometry>
-            <material name="black"/>
-        </visual>
-        <collision>
-            <geometry>
-                <cylinder radius="${wheel_rad}" length="${wheel_len}"/>
-            </geometry>
-            <material name="black"/>
-        </collision>
-        <xacro:inertial_cylinder mass="${wheel_mass}" length="${wheel_len}" radius="${wheel_rad}">
-            <origin xyz="0 0 0" rpy="0 0 0"/>
-        </xacro:inertial_cylinder>
-    </link>
-    <joint name="right_drive_wheel_joint" type="continuous">
-        <parent link="base_link"/>
-        <child link="left_drive_wheel"/>
-        <origin xyz="-${drive_wheel_x_off} -${drive_wheel_y_off} -${drive_wheel_z_off}" rpy="${pi/2} 0 0 "/>
-        <axis xyz="0 0 1"/>
-    </joint>
-    <link name="left_drive_wheel">
-        <visual>
-            <geometry>
-                <cylinder radius="${wheel_rad}" length="${wheel_len}"/>
-            </geometry>
-            <material name="black"/>
-        </visual>
-        <collision>
-            <geometry>
-                <cylinder radius="${wheel_rad}" length="${wheel_len}"/>
-            </geometry>
-            <material name="black"/>
-        </collision>
-        <xacro:inertial_cylinder mass="${wheel_mass}" length="${wheel_len}" radius="${wheel_rad}">
-            <origin xyz="0 0 0" rpy="0 0 0"/>
-        </xacro:inertial_cylinder>
-    </link>
-    <joint name="left_drive_wheel_joint" type="continuous">
-        <parent link="base_link"/>
-        <child link="right_drive_wheel"/>
-        <origin xyz="-${drive_wheel_x_off} ${drive_wheel_y_off} -${drive_wheel_z_off}" rpy="-${pi/2} 0 0 "/>
-        <axis xyz="0 0 -1"/>
-    </joint>
-   <!-- STEERING WHEELS -->
-    <xacro:property name="steer_wheel_x_off" value="0.235"/>
-    <xacro:property name="steer_wheel_y_off" value="0.52297"/>
-    <xacro:property name="steer_wheel_z_off" value="0.208"/>
-    <link name="right_steering_wheel">
-        <visual>
-            <geometry>
-                <cylinder radius="${wheel_rad}" length="${wheel_len}"/>
-            </geometry>
-            <material name="light_grey"/>
-        </visual>
-        <collision>
-            <geometry>
-                <cylinder radius="${wheel_rad}" length="${wheel_len}"/>
-            </geometry>
-            <material name="light_grey"/>
-        </collision>
-        <xacro:inertial_cylinder mass="${wheel_mass}" length="${wheel_len}" radius="${wheel_rad}">
-            <origin xyz="0 0 0" rpy="0 0 0"/>
-        </xacro:inertial_cylinder>
-    </link>
-    <joint name="right_steering_wheel_joint" type="continuous">
-        <parent link="base_link"/>
-        <child link="right_steering_wheel"/>
-        <origin xyz="${steer_wheel_x_off} -${steer_wheel_y_off} -${steer_wheel_z_off}" rpy="${pi/2} 0 0 "/>
-        <axis xyz="0 0 1"/>
-    </joint>
-    <link name="left_steering_wheel">
-        <visual>
-            <geometry>
-                <cylinder radius="${wheel_rad}" length="${wheel_len}"/>
-            </geometry>
-            <material name="light_grey"/>
-        </visual>
-        <collision>
-            <geometry>
-                <cylinder radius="${wheel_rad}" length="${wheel_len}"/>
-            </geometry>
-            <material name="light_grey"/>
-        </collision>
-        <xacro:inertial_cylinder mass="${wheel_mass}" length="${wheel_len}" radius="${wheel_rad}">
-            <origin xyz="0 0 0" rpy="0 0 0"/>
-        </xacro:inertial_cylinder>
-    </link>
-    <joint name="left_steering_wheel_joint" type="continuous">
-        <parent link="base_link"/>
-        <child link="left_steering_wheel"/>
-        <origin xyz="${steer_wheel_x_off} ${steer_wheel_y_off} -${steer_wheel_z_off}" rpy="-${pi/2} 0 0 "/>
-        <axis xyz="0 0 -1"/>
-    </joint>
-    <link name="mid_steering_wheel">
-        <visual>
-            <geometry>
-                <cylinder radius="${wheel_rad}" length="${wheel_len}"/>
-            </geometry>
-            <material name="light_grey"/>
-        </visual>
-        <collision>
-            <geometry>
-                <cylinder radius="${wheel_rad}" length="${wheel_len}"/>
-            </geometry>
-            <material name="light_grey"/>
-        </collision>
-        <xacro:inertial_cylinder mass="${wheel_mass}" length="${wheel_len}" radius="${wheel_rad}">
-            <origin xyz="0 0 0" rpy="0 0 0"/>
-        </xacro:inertial_cylinder>
-    </link>
-    <joint name="mid_steering_wheel_joint" type="continuous">
-        <parent link="base_link"/>
-        <child link="mid_steering_wheel"/>
-        <origin xyz="${steer_wheel_x_off} 0 -${steer_wheel_z_off}" rpy="-${pi/2} 0 0 "/>
-        <axis xyz="0 0 -1"/>
-    </joint>
-    <!-- SERVO -->
-    <xacro:property name="servo_x" value="0.05475"/>
-    <xacro:property name="servo_y" value="0.15"/>
-    <link name="servo">
-        <visual>
-            <geometry>
-                <cylinder radius="${wheel_rad}" length="${wheel_len}"/>
-            </geometry>
-            <material name="light_grey"/>
-        </visual>
-        <collision>
-            <geometry>
-                <cylinder radius="${wheel_rad}" length="${wheel_len}"/>
-            </geometry>
-            <material name="light_grey"/>
-        </collision>
-        <xacro:inertial_cylinder mass="${wheel_mass}" length="${wheel_len}" radius="${wheel_rad}">
-            <origin xyz="0 0 0" rpy="0 0 0"/>
-        </xacro:inertial_cylinder>
-    </link>
-    <joint name="servo_joint" type="continuous">
-        <parent link="base_link"/>
-        <child link="servo"/>
-        <origin xyz="${servo_x} ${servo_y} -${steer_wheel_z_off}" rpy="-${pi/2} 0 0 "/>
-        <axis xyz="0 0 -1"/>
-    </joint>
-    <!-- Adding colours to wheels for gazebo -->
-    <gazebo reference="left_drive_wheel">
-        <material>Gazebo/Black</material>
-    </gazebo>
-    <gazebo reference="right_drive_wheel">
-        <material>Gazebo/Black</material>
-    </gazebo>
-    <gazebo reference="left_steering_wheel">
-        <material>Gazebo/Black</material>
-    </gazebo>
-    <gazebo reference="right_steering_wheel">
-        <material>Gazebo/Black</material>
-    </gazebo>
 </robot>

Commit message: fix: lidar urdf fixed and positioned properly

File: esda_sim/description/esda.urdf.xacro (robot description, xacro)
@@ -5,5 +5,5 @@
     <xacro:include filename="esda_core.xacro"/>
     <xacro:include filename="wheels.xacro"/>
-    <!--<xacro:include filename="sensors/lidar.xacro"/>-->
+    <xacro:include filename="sensors/lidar.xacro"/>
     <xacro:include filename="sensors/piksi.xacro"/>
     <!--<xacro:include filename="sensors/camera.xacro"/>-->

File: esda_sim/description/sensors/lidar.xacro (robot description, xacro)
@@ -1,7 +1,71 @@
 <?xml version="1.0"?>
-<robot xmlns:xacro="http://www.ros.org/wiki/xacro">
-    <xacro:include filename="$(find velodyne_description)/urdf/VLP-16.urdf.xacro"/>
-    <VLP-16 parent="base_link" name="velodyne" topic="velodyne_points" hz="10" samples="440">
-        <origin xyz="0 0 1.7" rpy="0 0 0" />
-    </VLP-16>
+<robot xmlns:xacro="http://www.ros.org/wiki/xacro" name="VLP-16">
+    <xacro:property name="M_PI" value="3.1415926535897931" />
+    <xacro:property name="name" value="velodyne" />
+    <xacro:property name="parent" value="base_link" />
+    <xacro:property name="radius" value="0.0516" /> <!-- measured 50.5mm -->
+    <xacro:property name="height" value="0.0717" /> <!-- measured 72.8mm | top 14mm, mid 38.8mm, bottom 19mm-->
+    <xacro:property name="x" value="-0.149" />
+    <xacro:property name="y" value="0" />
+    <xacro:property name="z" value="0.5707" />
+    <joint name="${name}_base_mount_joint" type="fixed">
+        <origin xyz="${x} ${y} ${z}" rpy="0 0 0" />
+        <parent link="${parent}"/>
+        <child link="${name}_base_link"/>
+    </joint>
+    <link name="${name}_base_link">
+        <inertial>
+        <mass value="0.83"/>
+        <origin xyz="0 0 0.03585"/>
+        <inertia
+            ixx="${(0.83 * (3.0*0.0516*0.0516 + 0.0717*0.0717)) / 12.0}" ixy="0" ixz="0"
+            iyy="${(0.83 * (3.0*0.0516*0.0516 + 0.0717*0.0717)) / 12.0}" iyz="0"
+            izz="${0.5 * 0.83 * (0.0516*0.0516)}"/>
+        </inertial>
+        <!--
+        <visual>
+            <geometry>
+                <mesh filename="package://velodyne_description/meshes/VLP16_base_1.dae" />
+            </geometry>
+        </visual>
+        <visual>
+            <geometry>
+                <mesh filename="package://velodyne_description/meshes/VLP16_base_2.dae" />
+            </geometry>
+        </visual>
+        -->
+        <visual>
+            <origin rpy="0 0 0" xyz="0 0 0.03585"/>
+            <geometry>
+                <cylinder radius="${radius}" length="${height}"/>
+            </geometry>
+            <material name="light_grey"/>
+        </visual>
+        <collision>
+            <origin rpy="0 0 0" xyz="0 0 0.03585"/>
+            <geometry>
+                <cylinder radius="${radius}" length="${height}"/>
+            </geometry>
+        </collision>
+    </link>
+    <joint name="${name}_base_scan_joint" type="fixed" >
+        <origin xyz="0 0 0.0377" rpy="0 0 0" />
+        <parent link="${name}_base_link" />
+        <child link="${name}"/>
+    </joint>
+    <link name="${name}">
+	    <inertial>
+	        <mass value="0.01"/>
+	        <origin xyz="0 0 0"/>
+	        <inertia ixx="1e-7" ixy="0" ixz="0" iyy="1e-7" iyz="0" izz="1e-7"/>
+	    </inertial>
+	    <!--
+	    <visual>
+	        <origin xyz="0 0 -0.0377" />
+	        <geometry>
+	            <mesh filename="package://velodyne_description/meshes/VLP16_scan.dae" />
+	        </geometry>
+	    </visual>
+	    -->
+    </link>
 </robot>

File: esda_sim/description/steering_wheels.xacro (robot description, xacro)
@@ -114,4 +114,5 @@
     </joint>
     <!-- Define an arbitrary steering wheel as it's required for the AckermannControl plugin to work -->
+    <!--
     <link name="steering_wheel">
         <visual>
@@ -137,3 +138,4 @@
         <axis xyz="0 0 1"/>
     </joint>
+    -->
 </robot>

Commit message: refactoring launch files

File: esda_sim/description/esda.urdf.xacro (robot description, xacro)
@@ -8,4 +8,3 @@
     <xacro:include filename="sensors/piksi.xacro"/>
     <xacro:include filename="sensors/camera.xacro"/>
-    <xacro:include filename="control/ros2_control.xacro"/>
 </robot>

File: esda_sim/description/sensors/camera.xacro (robot description, xacro)
@@ -1,13 +1,8 @@
 <?xml version="1.0"?>
-<robot xmlns:xacro="http://www.ros.org/wiki/xacro" name="robot">
-    <xacro:arg name="camera_name"   default="zed2" />
-    <xacro:arg name="camera_model"  default="zed2" />
-    <xacro:property name="cam_p" value="0.646"/>
-    <xacro:include filename="$(find zed_wrapper)/urdf/zed_macro.urdf.xacro"/>
-    <xacro:zed_camera name="$(arg camera_name)" model="$(arg camera_model)"/>
-    <joint name="$(arg camera_name)_joint" type="fixed">
-        <parent link="base_link"/>
-        <child link="$(arg camera_name)_camera_link"/>
-        <origin xyz="0.271364 0.0 0.243727" rpy="0 ${cam_p} 0" />
-    </joint>
+<robot name="esda" xmlns:xacro="http://ros.org/wiki/xacro">
+  <joint name="zed_to_baselink" type="fixed">
+      <parent link="base_link"/>
+      <child link="zed_camera_link"/>
+      <origin xyz="0.271364 0.0 0.243727" rpy="0 0.646 0" />
+  </joint>
 </robot>

Commit message: launch bug fixes

File: esda_sim/description/esda.urdf.xacro (robot description, xacro)
@@ -8,4 +8,22 @@
     <xacro:include filename="sensors/piksi.xacro"/>
     <xacro:include filename="sensors/camera.xacro"/>
-    <xacro:include filename="control/gazebo_diff_control.xacro"/>
+    <!--<xacro:include filename="control/gazebo_diff_control.xacro"/>-->
+    <gazebo>
+        <plugin name="diff_drive" filename="libgazebo_ros_diff_drive.so">
+            <!-- Wheel Information -->
+            <left_joint>left_drive_wheel_joint</left_joint>
+            <right_joint>right_drive_wheel_joint</right_joint>
+            <wheel_separation>0.958</wheel_separation>
+            <wheel_diameter>0.265</wheel_diameter>
+            <!-- Limits -->
+            <max_wheel_torque>100</max_wheel_torque>
+            <max_wheel_acceleration>10.0</max_wheel_acceleration>
+            <!-- Output -->
+            <odometry_frame>odom</odometry_frame>
+            <robot_base_frame>base_link</robot_base_frame>
+            <publish_odom>true</publish_odom>
+            <publish_odom_tf>true</publish_odom_tf>
+            <publish_wheel_tf>true</publish_wheel_tf>
+        </plugin>
+    </gazebo>
 </robot>

File: esda_sim/description/sensors/camera.xacro (robot description, xacro)
@@ -1,4 +1,6 @@
 <?xml version="1.0"?>
 <robot name="esda" xmlns:xacro="http://ros.org/wiki/xacro">
+  <link name="zed_camera_link">
+  </link>
   <joint name="zed_to_baselink" type="fixed">
       <parent link="base_link"/>

Commit message: fixed urdf sensor outputs for sim

File: esda_sim/description/esda.urdf.xacro (robot description, xacro)
@@ -8,5 +8,4 @@
     <xacro:include filename="sensors/piksi.xacro"/>
     <xacro:include filename="sensors/camera.xacro"/>
-    <!--<xacro:include filename="control/gazebo_diff_control.xacro"/>-->
     <gazebo>
         <plugin name="diff_drive" filename="libgazebo_ros_diff_drive.so">

File: esda_sim/description/sensors/lidar.xacro (robot description, xacro)
@@ -60,14 +60,6 @@
 	        <inertia ixx="1e-7" ixy="0" ixz="0" iyy="1e-7" iyz="0" izz="1e-7"/>
 	    </inertial>
-	    <!--
-	    <visual>
-	        <origin xyz="0 0 -0.0377" />
-	        <geometry>
-	            <mesh filename="package://velodyne_description/meshes/VLP16_scan.dae" />
-	        </geometry>
-	    </visual>
-	    -->
     </link>
-    <gazebo reference="velodyne">
+    <gazebo reference="velodyne_base_link">
         <material>Gazebo/Grey</material>
         <sensor name="laser" type="ray">

File: esda_sim/description/sensors/piksi.xacro (robot description, xacro)
@@ -31,6 +31,6 @@
     </joint>
     <!-- Obtained from https://medium.com/@bytesrobotics/a-review-of-the-ros2-urdf-gazebo-sensor-91e947c633d7 -->
-    <gazebo reference="gps_link">
-        <sensor name="gps_sensor" type="gps">
+    <gazebo reference="swiftnav-gnss">
+        <sensor name="gps" type="gps">
             <always_on>true</always_on>
             <update_rate>1.0</update_rate>
@@ -45,6 +45,6 @@
         <material>Gazebo/Grey</material>
     </gazebo>
-    <gazebo reference="imu_link">
-        <sensor name="br_imu" type="imu">
+    <gazebo reference="swiftnav-gnss">
+        <sensor name="imu" type="imu">
             <always_on>true</always_on>
             <update_rate>100</update_rate>
@@ -93,6 +93,5 @@
             <plugin name="bytes_imu" filename="libgazebo_ros_imu_sensor.so">
                 <ros>
-                    <namespace>imu</namespace>
-                    <remapping>~/out:=data</remapping>
+                    <remapping>~/out:=imu</remapping>
                 </ros>
                 <initial_orientation_as_reference>false</initial_orientation_as_reference>
