Commit message: removed bakc caster from esda sim

File: esda_sim/description/caster_wheels.xacro (robot description, xacro)
@@ -44,5 +44,5 @@
         </xacro:inertial_sphere>
     </link>
-    <link name="back_caster">
+    <!--<link name="back_caster">
         <visual>
             <geometry>
@@ -60,5 +60,5 @@
             <origin xyz="0 0 0" rpy="0 0 0"/>
         </xacro:inertial_sphere>
-    </link>
+    </link>-->
     <!-- -->
     <joint name="right_caster_joint" type="fixed">
@@ -72,8 +72,8 @@
         <origin xyz="${caster_x + caster_x_off} ${caster_y} -${caster_z}" rpy="0 0 0 "/>
     </joint>
-    <joint name="back_caster_joint" type="fixed">
+    <!--<joint name="back_caster_joint" type="fixed">
         <parent link="base_link"/>
         <child link="back_caster"/>
         <origin xyz="-${caster_x/0.33} 0 -${caster_z}" rpy="0 0 0 "/>
-    </joint>
+    </joint>-->
 </robot>
