Commit message: feat: fronte wheels can now turn and spin in esda sim

File: esda_sim/description/control/ackermann_control.xacro (robot description, xacro)
@@ -11,6 +11,6 @@
                turning motion
           -->
-          <left_steering_joint>left_steering_wheel_joint</left_steering_joint>
-          <right_steering_joint>right_steering_wheel_joint</right_steering_joint>
+          <left_steering_joint>left_wheel_axle_joint</left_steering_joint>
+          <right_steering_joint>right_wheel_axle_joint</right_steering_joint>
           <!-- Must point to the front turning wheel joints that implement
                axle rotation

File: esda_sim/description/esda.urdf.xacro (robot description, xacro)
@@ -9,4 +9,4 @@
     <!--<xacro:include filename="camera.xacro"/>-->
     <!--<xacro:include filename="ackermann_control.xacro"/>-->
-    <xacro:include filename="diff_control.xacro"/>
+    <!-- <xacro:include filename="diff_control.xacro"/> -->
 </robot>

File: esda_sim/description/steering_wheels.xacro (robot description, xacro)
@@ -7,5 +7,5 @@
     <xacro:property name="steer_wheel_y_off" value="0.52297"/>
     <xacro:property name="steer_wheel_z_off" value="0.208"/>
-    <!-- Define the wheels that turn -->
+    <!-- Define the wheels that spin -->
     <link name="right_steering_wheel">
         <visual>
@@ -42,9 +42,9 @@
         </xacro:inertial_cylinder>
     </link>
-    <!-- Define the wheels that spin -->
-    <link name="right_axle_wheel">
+    <!-- Define the component that will turn around z which the wheels will attach to -->
+    <link name="right_steering_link">
         <visual>
             <geometry>
-                <cylinder radius="${wheel_rad}" length="${wheel_len}"/>
+                <sphere radius="0.01"/>
             </geometry>
             <material name="light_grey"/>
@@ -52,16 +52,16 @@
         <collision>
             <geometry>
-                <cylinder radius="${wheel_rad}" length="${wheel_len}"/>
+                <sphere radius="0.01"/>
             </geometry>
             <material name="light_grey"/>
         </collision>
-        <xacro:inertial_cylinder mass="${wheel_mass}" length="${wheel_len}" radius="${wheel_rad}">
+        <xacro:inertial_sphere mass="0" radius="0.01">
             <origin xyz="0 0 0" rpy="0 0 0"/>
-        </xacro:inertial_cylinder>
+        </xacro:inertial_sphere>
     </link>
-    <link name="left_axle_wheel">
+    <link name="left_steering_link">
         <visual>
             <geometry>
-                <cylinder radius="${wheel_rad}" length="${wheel_len}"/>
+                <sphere radius="0.01"/>
             </geometry>
             <material name="light_grey"/>
@@ -69,11 +69,11 @@
         <collision>
             <geometry>
-                <cylinder radius="${wheel_rad}" length="${wheel_len}"/>
+                <sphere radius="0.01"/>
             </geometry>
             <material name="light_grey"/>
         </collision>
-        <xacro:inertial_cylinder mass="${wheel_mass}" length="${wheel_len}" radius="${wheel_rad}">
+        <xacro:inertial_sphere mass="0" radius="0.01">
             <origin xyz="0 0 0" rpy="0 0 0"/>
-        </xacro:inertial_cylinder>
+        </xacro:inertial_sphere>
     </link>
     <!-- Note that in the following joint definitions, when defining the wheels
@@ -84,29 +84,31 @@
     <!-- Define the wheels rotation around the x axis so they can roll forward -->
     <joint name="right_wheel_axle_joint" type="continuous">
-        <parent link="base_link"/>
-        <child link="right_axle_wheel"/>
-        <origin xyz="${steer_wheel_x_off} -${steer_wheel_y_off} -${steer_wheel_z_off}" rpy="${pi/2} 0 0 "/>
+        <parent link="right_steering_link"/>
+        <child link="right_steering_wheel"/>
+        <origin xyz="0 0 0" rpy="0 0 0"/>
         <axis xyz="0 0 1"/>
     </joint>
     <joint name="left_wheel_axle_joint" type="continuous">
-        <parent link="base_link"/>
-        <child link="left_axle_wheel"/>
-        <origin xyz="${steer_wheel_x_off} ${steer_wheel_y_off} -${steer_wheel_z_off}" rpy="-${pi/2} 0 0 "/>
+        <parent link="left_steering_link"/>
+        <child link="left_steering_wheel"/>
+        <origin xyz="0 0 0" rpy="0 0 0 "/>
         <axis xyz="0 0 -1"/>
     </joint>
-    <!-- Define the wheels rotation around the z-axis so they can turn sideways -->
-    <joint name="right_steering_wheel_joint" type="revolute">
+    <!-- The steer_link will rotate around z-axis and because the wheels are jointed to this, their
+         position is relative to this and thus will follow the turn of the steer_link.
+    -->
+    <joint name="right_steer_joint" type="revolute">
         <parent link="base_link"/>
-        <child link="right_steering_wheel"/>
+        <child link="right_steering_link"/>
         <origin xyz="${steer_wheel_x_off} -${steer_wheel_y_off} -${steer_wheel_z_off}" rpy="${pi/2} 0 0 "/>
         <axis xyz="0 -1 0"/>
-        <limit lower="-${6/10}" upper="${6/10}" effort="1" velocity="1"/>
+        <limit effort="100" lower="-0.41" upper="0.41" velocity="0.5"/>
     </joint>
-    <joint name="left_steering_wheel_joint" type="revolute">
+    <joint name="left_steer_joint" type="revolute">
         <parent link="base_link"/>
-        <child link="left_steering_wheel"/>
+        <child link="left_steering_link"/>
         <origin xyz="${steer_wheel_x_off} ${steer_wheel_y_off} -${steer_wheel_z_off}" rpy="-${pi/2} 0 0 "/>
         <axis xyz="0 1 0"/>
-        <limit lower="-${6/10}" upper="${6/10}" effort="1" velocity="1"/>
+        <limit effort="100" lower="-0.41" upper="0.41" velocity="0.5"/>
     </joint>
     <!-- Define an arbitrary steering wheel as it's required for the AckermannControl plugin to work -->

Commit message: debugging sim issues with gazebo render

File: esda_sim/description/control/ackermann_control.xacro (robot description, xacro)
@@ -3,40 +3,42 @@
     <gazebo>
         <plugin name="gazebo_ros_ackermann_drive" filename="libgazebo_ros_ackermann_drive.so">
-          <update_rate>100.0</update_rate>
-          <!-- WHEELS -->
-          <!-- Must point to the rear drive wheel joints -->
-          <rear_left_joint>left_drive_wheel_joint</rear_left_joint>
-          <rear_right_joint>right_drive_wheel_joint</rear_right_joint>
-          <!-- Must point to the front turning wheel joints that implement
-               turning motion
-          -->
-          <left_steering_joint>left_wheel_axle_joint</left_steering_joint>
-          <right_steering_joint>right_wheel_axle_joint</right_steering_joint>
-          <!-- Must point to the front turning wheel joints that implement
-               axle rotation
-          -->
-          <front_left_joint>left_wheel_axle_joint</front_left_joint>
-          <front_right_joint>right_wheel_axle_joint</front_right_joint>
-          <!-- Arbitrary steering wheel to fulfil the API -->
-          <steering_wheel_joint>steering_wheel_joint</steering_wheel_joint>
-          <!-- Max absolute steer angle for tyre in radians TODO -->
-          <max_steer>0.6458</max_steer>
-          <!-- Max absolute steering angle of steering wheel TODO -->
-          <max_steering_angle>7.85</max_steering_angle>
-          <!-- Max absolute linear speed is 5 miles/h, converted here to m/s -->
-          <max_speed>2.2352</max_speed>
-          <!-- PID tuning -->
-          <left_steering_pid_gain>1500 0 1</left_steering_pid_gain>
-          <left_steering_i_range>0 0</left_steering_i_range>
-          <right_steering_pid_gain>1500 0 1</right_steering_pid_gain>
-          <right_steering_i_range>0 0</right_steering_i_range>
-          <linear_velocity_pid_gain>1000 0 1</linear_velocity_pid_gain>
-          <linear_velocity_i_range>0 0</linear_velocity_i_range>
-          <!-- Output -->
-          <odometry_frame>odom_demo</odometry_frame>
-          <robot_base_frame>base_link</robot_base_frame>
-          <publish_odom>true</publish_odom>
-          <publish_odom_tf>true</publish_odom_tf>
-          <publish_wheel_tf>true</publish_wheel_tf>
+            <ros>
+                <namespace>demo</namespace>
+                <remapping>cmd_vel:=cmd_demo</remapping>
+                <remapping>odom:=odom_demo</remapping>
+                <remapping>distance:=distance_demo</remapping>
+            </ros>
+            <update_rate>100.0</update_rate>
+            <!-- WHEELS -->
+            <!-- Drive wheel joints that implement rotation about x-axis -->
+            <rear_left_joint>left_drive_wheel_joint</rear_left_joint>
+            <rear_right_joint>right_drive_wheel_joint</rear_right_joint>
+            <!-- Turning wheel axis joints that implement rotation about x-axis -->
+            <left_steering_joint>left_steer_joint</left_steering_joint>
+            <right_steering_joint>right_steer_joint</right_steering_joint>
+            <!-- TUrning wheel joints that implement steering around z-axis -->
+            <front_left_joint>left_wheel_axle_joint</front_left_joint>
+            <front_right_joint>right_wheel_axle_joint</front_right_joint>
+            <!-- Arbitrary steering wheel to fulfil the API -->
+            <steering_wheel_joint>steering_wheel_joint</steering_wheel_joint>
+            <!-- Max absolute steer angle for tyre in radians TODO -->
+            <max_steer>0.6458</max_steer>
+            <!-- Max absolute steering angle of steering wheel TODO -->
+            <max_steering_angle>7.85</max_steering_angle>
+            <!-- Max absolute linear speed in m/s -->
+            <max_speed>10</max_speed>
+            <!-- PID tuning -->
+            <left_steering_pid_gain>1500 0 1</left_steering_pid_gain>
+            <left_steering_i_range>0 0</left_steering_i_range>
+            <right_steering_pid_gain>1500 0 1</right_steering_pid_gain>
+            <right_steering_i_range>0 0</right_steering_i_range>
+            <linear_velocity_pid_gain>1000 0 1</linear_velocity_pid_gain>
+            <linear_velocity_i_range>0 0</linear_velocity_i_range>
+            <!-- Output -->
+            <odometry_frame>odom_demo</odometry_frame>
+            <robot_base_frame>base_link</robot_base_frame>
+            <publish_odom>true</publish_odom>
+            <publish_odom_tf>true</publish_odom_tf>
+            <publish_wheel_tf>true</publish_wheel_tf>
         </plugin>
     </gazebo>

File: esda_sim/description/drive_wheels.xacro (robot description, xacro)
@@ -28,5 +28,5 @@
         <child link="left_drive_wheel"/>
         <origin xyz="-${drive_wheel_x_off} -${drive_wheel_y_off} -${drive_wheel_z_off}" rpy="${pi/2} 0 0 "/>
-        <axis xyz="0 0 1"/>
+        <axis xyz="0 0 -1"/>
     </joint>
     <link name="left_drive_wheel">
@@ -51,5 +51,5 @@
         <child link="right_drive_wheel"/>
         <origin xyz="-${drive_wheel_x_off} ${drive_wheel_y_off} -${drive_wheel_z_off}" rpy="-${pi/2} 0 0 "/>
-        <axis xyz="0 0 -1"/>
+        <axis xyz="0 0 1"/>
     </joint>
 </robot>

File: esda_sim/description/esda.urdf.xacro (robot description, xacro)
@@ -5,8 +5,7 @@
     <xacro:include filename="esda_core.xacro"/>
     <xacro:include filename="wheels.xacro"/>
-    <xacro:include filename="lidar.xacro"/>
+    <!--<xacro:include filename="lidar.xacro"/>-->
     <xacro:include filename="piksi.xacro"/>
     <!--<xacro:include filename="camera.xacro"/>-->
-    <!--<xacro:include filename="ackermann_control.xacro"/>-->
-    <!-- <xacro:include filename="diff_control.xacro"/> -->
+    <xacro:include filename="ackermann_control.xacro"/>
 </robot>

File: esda_sim/description/steering_wheels.xacro (robot description, xacro)
@@ -42,9 +42,9 @@
         </xacro:inertial_cylinder>
     </link>
-    <!-- Define the component that will turn around z which the wheels will attach to -->
+    <!-- Define the component that will turn around z-axis which the wheels will attach to -->
     <link name="right_steering_link">
         <visual>
             <geometry>
-                <sphere radius="0.01"/>
+                <sphere radius="0.07"/>
             </geometry>
             <material name="light_grey"/>
@@ -52,9 +52,9 @@
         <collision>
             <geometry>
-                <sphere radius="0.01"/>
+                <sphere radius="0.07"/>
             </geometry>
             <material name="light_grey"/>
         </collision>
-        <xacro:inertial_sphere mass="0" radius="0.01">
+        <xacro:inertial_sphere mass="0.5" radius="0.07">
             <origin xyz="0 0 0" rpy="0 0 0"/>
         </xacro:inertial_sphere>
@@ -63,5 +63,5 @@
         <visual>
             <geometry>
-                <sphere radius="0.01"/>
+                <sphere radius="0.07"/>
             </geometry>
             <material name="light_grey"/>
@@ -69,30 +69,18 @@
         <collision>
             <geometry>
-                <sphere radius="0.01"/>
+                <sphere radius="0.07"/>
             </geometry>
             <material name="light_grey"/>
         </collision>
-        <xacro:inertial_sphere mass="0" radius="0.01">
+        <xacro:inertial_sphere mass="0.5" radius="0.07">
             <origin xyz="0 0 0" rpy="0 0 0"/>
         </xacro:inertial_sphere>
     </link>
-    <!-- Note that in the following joint definitions, when defining the wheels
-         axis of rotation, it refers to the wheel links axis, not base_link as
+    <!-- Note that in the following joint definitions, when defining the
+         axis of rotation, it refers to the links axis, not base_link as
          the wheels have been rotated 90deg for correct positioning.
          The comments below however, are in reference to the base_link axis.
+         THe approach taken was sources from https://robotics.stackexchange.com/a/106022
     -->
-    <!-- Define the wheels rotation around the x axis so they can roll forward -->
-    <joint name="right_wheel_axle_joint" type="continuous">
-        <parent link="right_steering_link"/>
-        <child link="right_steering_wheel"/>
-        <origin xyz="0 0 0" rpy="0 0 0"/>
-        <axis xyz="0 0 1"/>
-    </joint>
-    <joint name="left_wheel_axle_joint" type="continuous">
-        <parent link="left_steering_link"/>
-        <child link="left_steering_wheel"/>
-        <origin xyz="0 0 0" rpy="0 0 0 "/>
-        <axis xyz="0 0 -1"/>
-    </joint>
     <!-- The steer_link will rotate around z-axis and because the wheels are jointed to this, their
          position is relative to this and thus will follow the turn of the steer_link.
@@ -103,5 +91,5 @@
         <origin xyz="${steer_wheel_x_off} -${steer_wheel_y_off} -${steer_wheel_z_off}" rpy="${pi/2} 0 0 "/>
         <axis xyz="0 -1 0"/>
-        <limit effort="100" lower="-0.41" upper="0.41" velocity="0.5"/>
+        <limit effort="100" lower="-0.41" upper="0.41" velocity="1"/>
     </joint>
     <joint name="left_steer_joint" type="revolute">
@@ -110,5 +98,18 @@
         <origin xyz="${steer_wheel_x_off} ${steer_wheel_y_off} -${steer_wheel_z_off}" rpy="-${pi/2} 0 0 "/>
         <axis xyz="0 1 0"/>
-        <limit effort="100" lower="-0.41" upper="0.41" velocity="0.5"/>
+        <limit effort="100" lower="-0.41" upper="0.41" velocity="1"/>
+    </joint>
+    <!-- Define the wheels rotation around the x axis so they can roll forward -->
+    <joint name="right_wheel_axle_joint" type="continuous">
+        <parent link="right_steering_link"/>
+        <child link="right_steering_wheel"/>
+        <origin xyz="0 0 0" rpy="0 0 0"/>
+        <axis xyz="0 0 -1"/>
+    </joint>
+    <joint name="left_wheel_axle_joint" type="continuous">
+        <parent link="left_steering_link"/>
+        <child link="left_steering_wheel"/>
+        <origin xyz="0 0 0" rpy="0 0 0 "/>
+        <axis xyz="0 0 1"/>
     </joint>
     <!-- Define an arbitrary steering wheel as it's required for the AckermannControl plugin to work -->

Commit message: urdf fixes

File: esda_sim/description/control/ackermann_control.xacro (robot description, xacro)
@@ -2,5 +2,5 @@
 <robot xmlns:xacro="http://www.ros.org/wiki/xacro">
     <gazebo>
-        <plugin name="gazebo_ros_ackermann_drive" filename="libgazebo_ros_ackermann_drive.so">
+        <plugin name="ackermann_drive" filename="libgazebo_ros_ackermann_drive.so">
             <ros>
                 <namespace>demo</namespace>

File: esda_sim/description/drive_wheels.xacro (robot description, xacro)
@@ -26,5 +26,5 @@
     <joint name="right_drive_wheel_joint" type="continuous">
         <parent link="base_link"/>
-        <child link="left_drive_wheel"/>
+        <child link="right_drive_wheel"/>
         <origin xyz="-${drive_wheel_x_off} -${drive_wheel_y_off} -${drive_wheel_z_off}" rpy="${pi/2} 0 0 "/>
         <axis xyz="0 0 -1"/>
@@ -49,5 +49,5 @@
     <joint name="left_drive_wheel_joint" type="continuous">
         <parent link="base_link"/>
-        <child link="right_drive_wheel"/>
+        <child link="left_drive_wheel"/>
         <origin xyz="-${drive_wheel_x_off} ${drive_wheel_y_off} -${drive_wheel_z_off}" rpy="-${pi/2} 0 0 "/>
         <axis xyz="0 0 1"/>

File: esda_sim/description/esda.urdf.xacro (robot description, xacro)
@@ -1,11 +1,11 @@
 <?xml version="1.0"?>
 <robot xmlns:xacro="http://www.ros.org/wiki/xacro" name="robot">
-    <xacro:include filename="inertial_macros.xacro"/>
-    <xacro:include filename="materials.xacro"/>
+    <xacro:include filename="util/inertial_macros.xacro"/>
+    <xacro:include filename="util/materials.xacro"/>
     <xacro:include filename="esda_core.xacro"/>
     <xacro:include filename="wheels.xacro"/>
-    <!--<xacro:include filename="lidar.xacro"/>-->
-    <xacro:include filename="piksi.xacro"/>
-    <!--<xacro:include filename="camera.xacro"/>-->
-    <xacro:include filename="ackermann_control.xacro"/>
+    <!--<xacro:include filename="sensors/lidar.xacro"/>-->
+    <xacro:include filename="sensors/piksi.xacro"/>
+    <!--<xacro:include filename="sensors/camera.xacro"/>-->
+    <xacro:include filename="control/ackermann_control.xacro"/>
 </robot>

File: esda_sim/description/steering_wheels.xacro (robot description, xacro)
@@ -46,5 +46,5 @@
         <visual>
             <geometry>
-                <sphere radius="0.07"/>
+                <cylinder radius="${wheel_rad}" length="${wheel_len}"/>
             </geometry>
             <material name="light_grey"/>
@@ -52,16 +52,16 @@
         <collision>
             <geometry>
-                <sphere radius="0.07"/>
+                <cylinder radius="${wheel_rad}" length="${wheel_len}"/>
             </geometry>
             <material name="light_grey"/>
         </collision>
-        <xacro:inertial_sphere mass="0.5" radius="0.07">
+        <xacro:inertial_cylinder mass="${wheel_mass}" length="${wheel_len}" radius="${wheel_rad}">
             <origin xyz="0 0 0" rpy="0 0 0"/>
-        </xacro:inertial_sphere>
+        </xacro:inertial_cylinder>
     </link>
     <link name="left_steering_link">
         <visual>
             <geometry>
-                <sphere radius="0.07"/>
+                <cylinder radius="${wheel_rad}" length="${wheel_len}"/>
             </geometry>
             <material name="light_grey"/>
@@ -69,11 +69,11 @@
         <collision>
             <geometry>
-                <sphere radius="0.07"/>
+                <cylinder radius="${wheel_rad}" length="${wheel_len}"/>
             </geometry>
             <material name="light_grey"/>
         </collision>
-        <xacro:inertial_sphere mass="0.5" radius="0.07">
+        <xacro:inertial_cylinder mass="${wheel_mass}" length="${wheel_len}" radius="${wheel_rad}">
             <origin xyz="0 0 0" rpy="0 0 0"/>
-        </xacro:inertial_sphere>
+        </xacro:inertial_cylinder>
     </link>
     <!-- Note that in the following joint definitions, when defining the
