Commit message: ackerman gazebo plugin seems to be working

File: esda_sim/description/control/gazebo_ackermann_control.xacro (robot description, xacro)
@@ -4,6 +4,6 @@
         <plugin name="ackermann_drive" filename="libgazebo_ros_ackermann_drive.so">
             <ros>
-                <namespace>demo</namespace>
-                <remapping>cmd_vel:=cmd_demo</remapping>
+                <namespace></namespace>
+                <remapping>cmd_vel:=cmd_vel</remapping>
                 <remapping>odom:=odom_demo</remapping>
                 <remapping>distance:=distance_demo</remapping>

File: esda_sim/description/esda.urdf.xacro (robot description, xacro)
@@ -8,4 +8,4 @@
     <xacro:include filename="sensors/piksi.xacro"/>
     <xacro:include filename="sensors/camera.xacro"/>
-    <xacro:include filename="control/ros2_control_ackermann.xacro"/>
+    <xacro:include filename="control/gazebo_ackermann_control.xacro"/>
 </robot>

File: esda_sim/description/steering_wheels.xacro (robot description, xacro)
@@ -114,9 +114,8 @@
     </joint>
     <!-- Define an arbitrary steering wheel as it's required for the AckermannControl plugin to work -->
-    <!--
     <link name="steering_wheel">
         <visual>
             <geometry>
-                <cylinder radius="${wheel_rad}" length="${wheel_len}"/>
+                <cylinder radius="0.1" length="0.1"/>
             </geometry>
             <material name="light_grey"/>
@@ -124,9 +123,9 @@
         <collision>
             <geometry>
-                <cylinder radius="${wheel_rad}" length="${wheel_len}"/>
+                <cylinder radius="0.1" length="0.1"/>
             </geometry>
             <material name="black"/>
         </collision>
-        <xacro:inertial_cylinder mass="${wheel_mass}" length="${wheel_len}" radius="${wheel_rad}">
+        <xacro:inertial_cylinder mass="0" length="0.1" radius="0.1">
             <origin xyz="0 0 0" rpy="0 0 0"/>
         </xacro:inertial_cylinder>
@@ -135,7 +134,6 @@
         <parent link="base_link"/>
         <child link="steering_wheel"/>
-        <origin xyz="0.5 0 0.5" rpy="${pi/2} 0 ${pi/2}"/>
+        <origin xyz="0.1 0 0.1" rpy="0 0 0"/>
         <axis xyz="0 0 1"/>
     </joint>
-    -->
 </robot>
