Commit message: fix: updated piksi multi position and dimensions

File: esda_sim/description/sensors/lidar.xacro (robot description, xacro)
@@ -1,60 +1,7 @@
 <?xml version="1.0"?>
 <robot xmlns:xacro="http://www.ros.org/wiki/xacro">
-    <xacro:property name="lidar_rad" value="0.0515"/>
-    <xacro:property name="lidar_len" value="0.072"/>
-    <link name="velodyne">
-        <visual>
-            <geometry>
-                <cylinder radius="${lidar_rad}" length="${lidar_len}"/>
-            </geometry>
-            <material name="orange"/>
-        </visual>
-        <collision>
-            <geometry>
-                <cylinder radius="${lidar_rad}" length="${lidar_len}"/>
-            </geometry>
-            <material name="orange"/>
-        </collision>
-        <xacro:inertial_cylinder mass="1" radius="${lidar_rad}" length="${lidar_len}">
-            <origin xyz="0 0 0" rpy="0 0 0"/>
-        </xacro:inertial_cylinder>
-    </link>
-    <joint name="velodyne_joint" type="fixed">
-        <parent link="base_link"/>
-        <child link="velodyne"/>
-        <origin xyz="0 0 0.5" rpy="0 0 0"/>
-    </joint>
-    <gazebo reference="velodyne">
-        <material>Gazebo/Grey</material>
-        <sensor name="laser" type="ray">
-            <pose> 0 0 0 0 0 0 </pose>
-            <visualize>false</visualize>
-            <update_rate>10</update_rate>
-            <ray>
-                <scan>
-                    <horizontal>
-                        <samples>360</samples>
-                        <min_angle>-3.14</min_angle>
-                        <max_angle>3.14</max_angle>
-                    </horizontal>
-                    <vertical>
-                        <samples>10</samples>
-                        <min_angle>-0.2</min_angle>
-                        <max_angle>0</max_angle>
-                    </vertical>
-                </scan>
-                <range>
-                    <min>0.3</min>
-                    <max>4.5</max>
-                </range>
-            </ray>
-            <plugin name="laser_controller" filename="libgazebo_ros_ray_sensor.so">
-                <ros>
-                    <argument>~/out:=velodyne_points</argument>
-                </ros>
-                <output_type>sensor_msgs/PointCloud2</output_type>
-                <frame_name>velodyne</frame_name>
-            </plugin>
-        </sensor>
-    </gazebo>
+    <xacro:include filename="$(find velodyne_description)/urdf/VLP-16.urdf.xacro"/>
+    <VLP-16 parent="base_link" name="velodyne" topic="velodyne_points" hz="10" samples="440">
+        <origin xyz="0 0 1.7" rpy="0 0 0" />
+    </VLP-16>
 </robot>

File: esda_sim/description/sensors/piksi.xacro (robot description, xacro)
@@ -1,4 +1,9 @@
 <?xml version="1.0"?>
 <robot xmlns:xacro="http://www.ros.org/wiki/xacro">
+    <xacro:property name="width" value="0.11"/>
+    <xacro:property name="height" value="0.017"/>
+    <xacro:property name="x" value="-0.0223"/>
+    <xacro:property name="y" value="0.0563"/>
+    <xacro:property name="z" value="-0.0804"/>
     <!-- verify that the X and Y dimensions are placed in the right axis
     -->
@@ -6,5 +11,5 @@
         <visual>
             <geometry>
-                <box size="0.14 0.12 0.04"/>
+                <box size="${width} ${width} ${height}"/>
             </geometry>
             <material name="orange"/>
@@ -12,9 +17,9 @@
         <collision>
             <geometry>
-                <box size="0.14 0.12 0.04"/>
+                <box size="${width} ${width} ${height}"/>
             </geometry>
             <material name="orange"/>
         </collision>
-        <xacro:inertial_box mass="5" x="0.14" y="0.12" z="0.04">
+        <xacro:inertial_box mass="0" x="${width}" y="${width}" z="${height}">
             <origin xyz="0 0 0" rpy="0 0 0"/>
         </xacro:inertial_box>
@@ -23,5 +28,5 @@
         <parent link="base_link"/>
         <child link="swiftnav-gnss"/>
-        <origin xyz="0.35 0 0.1" rpy="0 0 0"/>
+        <origin xyz="${x} ${y} ${z}" rpy="0 0 0"/>
     </joint>
 </robot>

Commit message: feat: added gazebo scan plugin back to lidar urdf

File: esda_sim/description/sensors/lidar.xacro (robot description, xacro)
@@ -69,3 +69,36 @@
 	    -->
     </link>
+    <gazebo reference="velodyne">
+        <material>Gazebo/Grey</material>
+        <sensor name="laser" type="ray">
+            <pose> 0 0 0 0 0 0 </pose>
+            <visualize>false</visualize>
+            <update_rate>10</update_rate>
+            <ray>
+                <scan>
+                    <horizontal>
+                        <samples>360</samples>
+                        <min_angle>-3.14</min_angle>
+                        <max_angle>3.14</max_angle>
+                    </horizontal>
+                    <vertical>
+                        <samples>10</samples>
+                        <min_angle>-0.2</min_angle>
+                        <max_angle>0</max_angle>
+                    </vertical>
+                </scan>
+                <range>
+                    <min>0.3</min>
+                    <max>4.5</max>
+                </range>
+            </ray>
+            <plugin name="laser_controller" filename="libgazebo_ros_ray_sensor.so">
+                <ros>
+                    <argument>~/out:=velodyne_points</argument>
+                </ros>
+                <output_type>sensor_msgs/PointCloud2</output_type>
+                <frame_name>velodyne</frame_name>
+            </plugin>
+        </sensor>
+    </gazebo>
 </robot>
