Commit message: updated camera urdf, switched parent and child

File: esda_sim/description/sensors/camera.xacro (robot description, xacro)
@@ -6,6 +6,6 @@
     <xacro:zed_camera name="$(arg camera_name)" model="$(arg camera_model)"/>
     <joint name="$(arg camera_name)_joint" type="fixed">
-        <parent link="$(arg camera_name)_camera_link"/>
-        <child link="base_link"/>
+        <parent link="base_link"/>
+        <child link="$(arg camera_name)_camera_link"/>
         <origin xyz="-1 0.0 -0.35" py="0 -0.5 0" />
     </joint>

Commit message: updated repos pointer for zed to mcav fork

File: esda_sim/description/sensors/camera.xacro (robot description, xacro)
@@ -8,5 +8,5 @@
         <parent link="base_link"/>
         <child link="$(arg camera_name)_camera_link"/>
-        <origin xyz="-1 0.0 -0.35" py="0 -0.5 0" />
+        <origin xyz="1 0.0 0.35" py="0 -0.5 0" />
     </joint>
 </robot>

Commit message: Update camera.xacro positions

File: esda_sim/description/sensors/camera.xacro (robot description, xacro)
@@ -8,5 +8,5 @@
         <parent link="base_link"/>
         <child link="$(arg camera_name)_camera_link"/>
-        <origin xyz="1 0.0 0.35" py="0 -0.5 0" />
+        <origin xyz="0.271364 0.0 0.243727" rpy="0 -0.646 0" />
     </joint>
 </robot>

Commit message: fixed launch issues and XML tags for esda_sim

File: esda_sim/description/sensors/camera.xacro (robot description, xacro)
@@ -3,4 +3,5 @@
     <xacro:arg name="camera_name"   default="zed2" />
     <xacro:arg name="camera_model"  default="zed2" />
+    <xacro:property name="cam_p" value="0.646"/>
     <xacro:include filename="$(find zed_wrapper)/urdf/zed_macro.urdf.xacro"/>
     <xacro:zed_camera name="$(arg camera_name)" model="$(arg camera_model)"/>
@@ -8,5 +9,5 @@
         <parent link="base_link"/>
         <child link="$(arg camera_name)_camera_link"/>
-        <origin xyz="0.271364 0.0 0.243727" rpy="0 -0.646 0" />
+        <origin xyz="0.271364 0.0 0.243727" rpy="0 ${cam_p} 0" />
     </joint>
 </robot>
