Commit message: Added ros2_control_demo files

File: esda_ros2_control/diff_drive_asterius_hardware_interface/description/urdf/diffbot.urdf.xacro (robot description, xacro)
@@ -4,9 +4,9 @@
   <xacro:arg name="prefix" default="" />
   <xacro:arg name="use_mock_hardware" default="false" />
-  <xacro:include filename="$(find ros2_control_demo_description)/share/diff_drive_asterius_hardware_interface/urdf/diffbot_description.urdf.xacro" />
+  <xacro:include filename="$(find diff_drive_asterius_hardware_interface)/description/urdf/diffbot_description.urdf.xacro" />
   <!-- Import Rviz colors -->
-  <xacro:include filename="$(find ros2_control_demo_description)/share/diff_drive_asterius_hardware_interface/urdf/diffbot.materials.xacro" />
+  <xacro:include filename="$(find diff_drive_asterius_hardware_interface)/description/urdf/diffbot.materials.xacro" />
   <!-- Import diffbot ros2_control description -->
-  <xacro:include filename="$(find ros2_control_demo_example_2)/ros2_control/diffbot.ros2_control.xacro" />
+  <xacro:include filename="$(find diff_drive_asterius_hardware_interface)/description/ros2_control/diffbot.ros2_control.xacro" />
   <xacro:diffbot prefix="$(arg prefix)" />
   <xacro:diffbot_ros2_control

File: install/esda_sim/share/esda_sim/description/control/gazebo_ackermann_control.xacro (robot description, xacro)
@@ -1,45 +1 @@
-<?xml version="1.0"?>
-<robot xmlns:xacro="http://www.ros.org/wiki/xacro">
-    <gazebo>
-        <plugin name="ackermann_drive" filename="libgazebo_ros_ackermann_drive.so">
-            <ros>
-                <namespace></namespace>
-                <remapping>cmd_vel:=cmd_vel</remapping>
-                <remapping>odom:=odom_demo</remapping>
-                <remapping>distance:=distance_demo</remapping>
-            </ros>
-            <update_rate>100.0</update_rate>
-            <!-- WHEELS -->
-            <!-- Drive wheel joints that implement rotation about x-axis -->
-            <rear_left_joint>left_drive_wheel_joint</rear_left_joint>
-            <rear_right_joint>right_drive_wheel_joint</rear_right_joint>
-            <!-- Turning wheel axis joints that implement rotation about x-axis -->
-            <left_steering_joint>left_steer_joint</left_steering_joint>
-            <right_steering_joint>right_steer_joint</right_steering_joint>
-            <!-- TUrning wheel joints that implement steering around z-axis -->
-            <front_left_joint>left_wheel_axle_joint</front_left_joint>
-            <front_right_joint>right_wheel_axle_joint</front_right_joint>
-            <!-- Arbitrary steering wheel to fulfil the API -->
-            <steering_wheel_joint>steering_wheel_joint</steering_wheel_joint>
-            <!-- Max absolute steer angle for tyre in radians TODO -->
-            <max_steer>0.6458</max_steer>
-            <!-- Max absolute steering angle of steering wheel TODO -->
-            <max_steering_angle>7.85</max_steering_angle>
-            <!-- Max absolute linear speed in m/s -->
-            <max_speed>10</max_speed>
-            <!-- PID tuning -->
-            <left_steering_pid_gain>1500 0 1</left_steering_pid_gain>
-            <left_steering_i_range>0 0</left_steering_i_range>
-            <right_steering_pid_gain>1500 0 1</right_steering_pid_gain>
-            <right_steering_i_range>0 0</right_steering_i_range>
-            <linear_velocity_pid_gain>1000 0 1</linear_velocity_pid_gain>
-            <linear_velocity_i_range>0 0</linear_velocity_i_range>
-            <!-- Output -->
-            <odometry_frame>odom_demo</odometry_frame>
-            <robot_base_frame>base_link</robot_base_frame>
-            <publish_odom>true</publish_odom>
-            <publish_odom_tf>true</publish_odom_tf>
-            <publish_wheel_tf>true</publish_wheel_tf>
-        </plugin>
-    </gazebo>
-</robot>
+/home/samue/GitHub/ESDA/build/esda_sim/description/control/gazebo_ackermann_control.xacro

File: install/esda_sim/share/esda_sim/description/control/gazebo_diff_control.xacro (robot description, xacro)
@@ -1,21 +1 @@
-<?xml version="1.0"?>
-<robot xmlns:xacro="http://www.ros.org/wiki/xacro">
-    <gazebo>
-        <plugin name="diff_drive" filename="libgazebo_ros_diff_drive.so">
-            <!-- Wheel Information -->
-            <left_joint>left_drive_wheel_joint</left_joint>
-            <right_joint>right_drive_wheel_joint</right_joint>
-            <wheel_separation>0.958</wheel_separation>
-            <wheel_diameter>0.265</wheel_diameter>
-            <!-- Limits -->
-            <max_wheel_torque>100</max_wheel_torque>
-            <max_wheel_acceleration>10.0</max_wheel_acceleration>
-            <!-- Output -->
-            <odometry_frame>odom</odometry_frame>
-            <robot_base_frame>base_link</robot_base_frame>
-            <publish_odom>true</publish_odom>
-            <publish_odom_tf>true</publish_odom_tf>
-            <publish_wheel_tf>true</publish_wheel_tf>
-        </plugin>
-    </gazebo>
-</robot>
+/home/samue/GitHub/ESDA/build/esda_sim/description/control/gazebo_diff_control.xacro

File: install/esda_sim/share/esda_sim/description/control/ros2_control.xacro (robot description, xacro)
@@ -1,62 +1 @@
-<?xml version="1.0"?>
-<robot xmlns:xacro="http://www.ros.org/wiki/xacro">
-    <!-- TODO: determine min/max steer -->
-    <xacro:property name="steer_min" value="-45"/>
-    <xacro:property name="steer_max" value="45"/>
-    <!-- TODO: determine min/max vel -->
-    <xacro:property name="vel_min" value="0"/>
-    <xacro:property name="vel_max" value="10"/>
-    <ros2_control name="GazeboSystem" type="system">
-        <!-- Refer to the following link for more details on setting up R2C for gazebo sims
-            https://github.com/ros-controls/ros2_control_demos/blob/humble/example_9/description/ros2_control/rrbot.ros2_control.xacro
-        -->
-        <hardware>
-            <plugin>gazebo_ros2_control/GazeboSystem</plugin>
-        </hardware>
-        <!-- JOINT CONFIGURATIONS
-                <command_inteface> configures the commands we send
-                <state_interface> indicates what readings we want to get
-        -->
-        <!-- STEER WHEELS -->
-        <joint name="right_steer_joint">
-            <command_interface name="position">
-                <param name="min">${steer_min}</param>
-                <param name="max">${steer_max}</param>
-            </command_interface>
-            <state_interface name="position"/>
-        </joint>
-        <joint name="left_steer_joint">
-            <command_interface name="position">
-                <param name="min">${steer_min}</param>
-                <param name="max">${steer_max}</param>
-            </command_interface>
-            <state_interface name="position"/>
-        </joint>
-        <!-- DRIVE WHEELS -->
-        <joint name="right_drive_wheel_joint">
-            <command_interface name="velocity">
-                <param name="min">${vel_min}</param>
-                <param name="max">${vel_max}</param>
-            </command_interface>
-            <state_interface name="position"/>
-            <state_interface name="velocity"/>
-        </joint>
-        <joint name="left_drive_wheel_joint">
-            <command_interface name="velocity">
-                <param name="min">${vel_min}</param>
-                <param name="max">${vel_max}</param>
-            </command_interface>
-            <state_interface name="position"/>
-            <state_interface name="velocity"/>
-        </joint>
-    </ros2_control>
-    <!-- Tell Gazebo to ue R2C. This also has its own control manager.
-        Need to tell its manager where the config for the controllers is. Taken from  the following link
-        https://github.com/joshnewans/articubot_one/blob/0085689ee023baac604268cdf7a9ce85a0ed7bae/description/ros2_control.xacro
-    -->
-    <gazebo>
-        <plugin name="gazebo_ros2_control" filename="libgazebo_ros2_control.so">
-            <parameters>$(find esda_sim)/config/ros2_control_config.yaml</parameters>
-        </plugin>
-    </gazebo>
-</robot>
+/home/samue/GitHub/ESDA/build/esda_sim/description/control/ros2_control.xacro

File: install/esda_sim/share/esda_sim/description/drive_wheels.xacro (robot description, xacro)
@@ -1,55 +1 @@
-<?xml version="1.0"?>
-<robot xmlns:xacro="http://www.ros.org/wiki/xacro">
-    <!-- DRIVE WHEELS
-         Defines the 2 rear drive wheels that provide motion in the x-axis (forward motion).
-    -->
-    <xacro:property name="drive_wheel_x_off" value="0.38724"/>
-    <xacro:property name="drive_wheel_y_off" value="0.48166"/>
-    <xacro:property name="drive_wheel_z_off" value="0.22"/>
-    <link name="right_drive_wheel">
-        <visual>
-            <geometry>
-                <cylinder radius="${wheel_rad}" length="${wheel_len}"/>
-            </geometry>
-            <material name="black"/>
-        </visual>
-        <collision>
-            <geometry>
-                <cylinder radius="${wheel_rad}" length="${wheel_len}"/>
-            </geometry>
-            <material name="black"/>
-        </collision>
-        <xacro:inertial_cylinder mass="${wheel_mass}" length="${wheel_len}" radius="${wheel_rad}">
-            <origin xyz="0 0 0" rpy="0 0 0"/>
-        </xacro:inertial_cylinder>
-    </link>
-    <joint name="right_drive_wheel_joint" type="continuous">
-        <parent link="base_link"/>
-        <child link="right_drive_wheel"/>
-        <origin xyz="-${drive_wheel_x_off} -${drive_wheel_y_off} -${drive_wheel_z_off}" rpy="${pi/2} 0 0 "/>
-        <axis xyz="0 0 -1"/>
-    </joint>
-    <link name="left_drive_wheel">
-        <visual>
-            <geometry>
-                <cylinder radius="${wheel_rad}" length="${wheel_len}"/>
-            </geometry>
-            <material name="black"/>
-        </visual>
-        <collision>
-            <geometry>
-                <cylinder radius="${wheel_rad}" length="${wheel_len}"/>
-            </geometry>
-            <material name="black"/>
-        </collision>
-        <xacro:inertial_cylinder mass="${wheel_mass}" length="${wheel_len}" radius="${wheel_rad}">
-            <origin xyz="0 0 0" rpy="0 0 0"/>
-        </xacro:inertial_cylinder>
-    </link>
-    <joint name="left_drive_wheel_joint" type="continuous">
-        <parent link="base_link"/>
-        <child link="left_drive_wheel"/>
-        <origin xyz="-${drive_wheel_x_off} ${drive_wheel_y_off} -${drive_wheel_z_off}" rpy="-${pi/2} 0 0 "/>
-        <axis xyz="0 0 1"/>
-    </joint>
-</robot>
+/home/samue/GitHub/ESDA/build/esda_sim/description/drive_wheels.xacro

File: install/esda_sim/share/esda_sim/description/esda.urdf.xacro (robot description, xacro)
@@ -1,28 +1 @@
-<?xml version="1.0"?>
-<robot xmlns:xacro="http://www.ros.org/wiki/xacro" name="esda">
-    <xacro:include filename="util/inertial_macros.xacro"/>
-    <xacro:include filename="util/materials.xacro"/>
-    <xacro:include filename="esda_core.xacro"/>
-    <xacro:include filename="wheels.xacro"/>
-    <xacro:include filename="sensors/lidar.xacro"/>
-    <xacro:include filename="sensors/piksi.xacro"/>
-    <xacro:include filename="sensors/camera.xacro"/>
-    <gazebo>
-        <plugin name="diff_drive" filename="libgazebo_ros_diff_drive.so">
-            <!-- Wheel Information -->
-            <left_joint>left_drive_wheel_joint</left_joint>
-            <right_joint>right_drive_wheel_joint</right_joint>
-            <wheel_separation>0.958</wheel_separation>
-            <wheel_diameter>0.265</wheel_diameter>
-            <!-- Limits -->
-            <max_wheel_torque>100</max_wheel_torque>
-            <max_wheel_acceleration>10.0</max_wheel_acceleration>
-            <!-- Output -->
-            <odometry_frame>odom</odometry_frame>
-            <robot_base_frame>base_link</robot_base_frame>
-            <publish_odom>true</publish_odom>
-            <publish_odom_tf>true</publish_odom_tf>
-            <publish_wheel_tf>true</publish_wheel_tf>
-        </plugin>
-    </gazebo>
-</robot>
+/home/samue/GitHub/ESDA/build/esda_sim/description/esda.urdf.xacro

File: install/esda_sim/share/esda_sim/description/esda_core.xacro (robot description, xacro)
@@ -1,75 +1 @@
-<?xml version="1.0"?>
-<robot xmlns:xacro="http://www.ros.org/wiki/xacro">
-    <!-- ROOT LINK
-         the datum point/point of reference and point that
-         everything ultimately connects to
-    -->
-    <link name="base_link"></link>
-    <!-- base_footprint is a child but of base_link but
-         has the same position as its needed for SLAM toolbox
-    -->
-    <link name="base_footprint"></link>
-    <joint name="base_footprint_joint" type="fixed">
-        <parent link="base_link"/>
-        <child link="base_footprint"/>
-        <origin xyz="0 0 0"/>
-    </joint>
-    <!-- BODY LINKS
-         these define the body of the ESDA which is simplified
-         as a series of boxes
-    -->
-    <!-- DRIVE BOX LINK -->
-    <xacro:property name="drive_box_x" value="0.5725"/>
-    <xacro:property name="drive_box_y" value="0.575"/>
-    <xacro:property name="drive_box_z" value="0.276"/>
-    <xacro:property name="drive_box_m" value="35"/>
-    <link name="drive_box">
-        <visual>
-            <geometry>
-                <box size="${drive_box_x} ${drive_box_y} ${drive_box_z}" />
-            </geometry>
-            <material name="white"/>
-        </visual>
-        <collision>
-            <geometry>
-                <box size="${drive_box_x} ${drive_box_y} ${drive_box_z}" />
-            </geometry>
-            <material name="white"/>
-        </collision>
-        <xacro:inertial_box mass="${drive_box_m}" x="${drive_box_x}" y="${drive_box_y}" z="${drive_box_z}">
-            <origin xyz="0 0 0" rpy="0 0 0"/>
-        </xacro:inertial_box>
-    </link>
-    <joint name="drive_box_joint" type="fixed">
-        <parent link="base_link"/>
-        <child link="drive_box"/>
-        <origin xyz="-${drive_box_x/2} 0 0"/>
-    </joint>
-    <!-- STEERING BOX LINK -->
-    <xacro:property name="steer_box_x" value="0.378"/>
-    <xacro:property name="steer_box_y" value="0.575"/>
-    <xacro:property name="steer_box_z" value="0.146"/>
-    <xacro:property name="steer_box_m" value="29"/>
-    <link name="steering_box">
-        <visual>
-            <geometry>
-                <box size="${steer_box_x} ${steer_box_y} ${steer_box_z}" />
-            </geometry>
-            <material name="white"/>
-        </visual>
-        <collision>
-            <geometry>
-                <box size="${steer_box_x} ${steer_box_y} ${steer_box_z}" />
-            </geometry>
-            <material name="white"/>
-        </collision>
-        <xacro:inertial_box mass="${steer_box_m}" x="${steer_box_x}" y="${steer_box_y}" z="${steer_box_z}">
-            <origin xyz="0 0 0" rpy="0 0 0"/>
-        </xacro:inertial_box>
-    </link>
-    <joint name="steering_box_joint" type="fixed">
-        <parent link="base_link"/>
-        <child link="steering_box"/>
-        <origin xyz="${steer_box_x/2} 0 -${drive_box_z/2-steer_box_z/2}"/> <!-- -0.065 -->
-    </joint>
-</robot>
+/home/samue/GitHub/ESDA/build/esda_sim/description/esda_core.xacro

File: install/esda_sim/share/esda_sim/description/sensors/camera.xacro (robot description, xacro)
@@ -1,10 +1 @@
-<?xml version="1.0"?>
-<robot name="esda" xmlns:xacro="http://ros.org/wiki/xacro">
-  <link name="zed_camera_link">
-  </link>
-  <joint name="zed_to_baselink" type="fixed">
-      <parent link="base_link"/>
-      <child link="zed_camera_link"/>
-      <origin xyz="0.271364 0.0 0.243727" rpy="0 0.646 0" />
-  </joint>
-</robot>
+/home/samue/GitHub/ESDA/build/esda_sim/description/sensors/camera.xacro

File: install/esda_sim/share/esda_sim/description/sensors/lidar.xacro (robot description, xacro)
@@ -1,96 +1 @@
-<?xml version="1.0"?>
-<robot xmlns:xacro="http://www.ros.org/wiki/xacro" name="VLP-16">
-    <xacro:property name="M_PI" value="3.1415926535897931" />
-    <xacro:property name="name" value="velodyne" />
-    <xacro:property name="parent" value="base_link" />
-    <xacro:property name="radius" value="0.0516" /> <!-- measured 50.5mm -->
-    <xacro:property name="height" value="0.0717" /> <!-- measured 72.8mm | top 14mm, mid 38.8mm, bottom 19mm-->
-    <xacro:property name="x" value="-0.149" />
-    <xacro:property name="y" value="0" />
-    <xacro:property name="z" value="0.5707" />
-    <joint name="${name}_base_mount_joint" type="fixed">
-        <origin xyz="${x} ${y} ${z}" rpy="0 0 0" />
-        <parent link="${parent}"/>
-        <child link="${name}_base_link"/>
-    </joint>
-    <link name="${name}_base_link">
-        <inertial>
-        <mass value="0.83"/>
-        <origin xyz="0 0 0.03585"/>
-        <inertia
-            ixx="${(0.83 * (3.0*0.0516*0.0516 + 0.0717*0.0717)) / 12.0}" ixy="0" ixz="0"
-            iyy="${(0.83 * (3.0*0.0516*0.0516 + 0.0717*0.0717)) / 12.0}" iyz="0"
-            izz="${0.5 * 0.83 * (0.0516*0.0516)}"/>
-        </inertial>
-        <!--
-        <visual>
-            <geometry>
-                <mesh filename="package://velodyne_description/meshes/VLP16_base_1.dae" />
-            </geometry>
-        </visual>
-        <visual>
-            <geometry>
-                <mesh filename="package://velodyne_description/meshes/VLP16_base_2.dae" />
-            </geometry>
-        </visual>
-        -->
-        <visual>
-            <origin rpy="0 0 0" xyz="0 0 0.03585"/>
-            <geometry>
-                <cylinder radius="${radius}" length="${height}"/>
-            </geometry>
-            <material name="light_grey"/>
-        </visual>
-        <collision>
-            <origin rpy="0 0 0" xyz="0 0 0.03585"/>
-            <geometry>
-                <cylinder radius="${radius}" length="${height}"/>
-            </geometry>
-        </collision>
-    </link>
-    <joint name="${name}_base_scan_joint" type="fixed" >
-        <origin xyz="0 0 0.0377" rpy="0 0 0" />
-        <parent link="${name}_base_link" />
-        <child link="${name}"/>
-    </joint>
-    <link name="${name}">
-	    <inertial>
-	        <mass value="0.01"/>
-	        <origin xyz="0 0 0"/>
-	        <inertia ixx="1e-7" ixy="0" ixz="0" iyy="1e-7" iyz="0" izz="1e-7"/>
-	    </inertial>
-    </link>
-    <gazebo reference="velodyne_base_link">
-        <material>Gazebo/Grey</material>
-        <sensor name="laser" type="ray">
-            <pose> 0 0 0 0 0 0 </pose>
-            <visualize>false</visualize>
-            <update_rate>10</update_rate>
-            <ray>
-                <scan>
-                    <horizontal>
-                        <samples>360</samples>
-                        <min_angle>-3.14</min_angle>
-                        <max_angle>3.14</max_angle>
-                    </horizontal>
-                    <vertical>
-                        <samples>10</samples>
-                        <min_angle>-0.2</min_angle>
-                        <max_angle>0</max_angle>
-                    </vertical>
-                </scan>
-                <range>
-                    <min>0.3</min>
-                    <max>4.5</max>
-                </range>
-            </ray>
-            <plugin name="laser_controller" filename="libgazebo_ros_ray_sensor.so">
-                <ros>
-                    <argument>~/out:=velodyne_points</argument>
-                </ros>
-                <output_type>sensor_msgs/PointCloud2</output_type>
-                <frame_name>velodyne</frame_name>
-            </plugin>
-        </sensor>
-    </gazebo>
-</robot>
+/home/samue/GitHub/ESDA/build/esda_sim/description/sensors/lidar.xacro
