Commit message: Added ros2_control_demo files

File: install/esda_sim/share/esda_sim/description/sensors/piksi.xacro (robot description, xacro)
@@ -1,101 +1 @@
-<?xml version="1.0"?>
-<robot xmlns:xacro="http://www.ros.org/wiki/xacro">
-    <xacro:property name="width" value="0.11"/>
-    <xacro:property name="height" value="0.017"/>
-    <xacro:property name="x" value="-0.0223"/>
-    <xacro:property name="y" value="0.0563"/>
-    <xacro:property name="z" value="-0.0804"/>
-    <!-- verify that the X and Y dimensions are placed in the right axis
-    -->
-    <link name="swiftnav-gnss">
-        <visual>
-            <geometry>
-                <box size="${width} ${width} ${height}"/>
-            </geometry>
-            <material name="orange"/>
-        </visual>
-        <collision>
-            <geometry>
-                <box size="${width} ${width} ${height}"/>
-            </geometry>
-            <material name="orange"/>
-        </collision>
-        <xacro:inertial_box mass="0" x="${width}" y="${width}" z="${height}">
-            <origin xyz="0 0 0" rpy="0 0 0"/>
-        </xacro:inertial_box>
-    </link>
-    <joint name="swiftnav_joint" type="fixed">
-        <parent link="base_link"/>
-        <child link="swiftnav-gnss"/>
-        <origin xyz="${x} ${y} ${z}" rpy="0 0 0"/>
-    </joint>
-    <!-- Obtained from https://medium.com/@bytesrobotics/a-review-of-the-ros2-urdf-gazebo-sensor-91e947c633d7 -->
-    <gazebo reference="swiftnav-gnss">
-        <sensor name="gps" type="gps">
-            <always_on>true</always_on>
-            <update_rate>1.0</update_rate>
-            <plugin name="gps_controller" filename="libgazebo_ros_gps_sensor.so">
-                <ros>
-                    <!-- <namespace>/br</namespace> -->
-                    <remapping>gps_controller/out:=navsatfix</remapping>
-                </ros>
-                <frame_name>piksi</frame_name>
-            </plugin>
-        </sensor>
-        <material>Gazebo/Grey</material>
-    </gazebo>
-    <gazebo reference="swiftnav-gnss">
-        <sensor name="imu" type="imu">
-            <always_on>true</always_on>
-            <update_rate>100</update_rate>
-            <imu>
-            <angular_velocity>
-                <x>
-                <noise type="gaussian">
-                    <mean>0.0</mean>
-                    <stddev>2e-4</stddev>
-                </noise>
-                </x>
-                <y>
-                <noise type="gaussian">
-                    <mean>0.0</mean>
-                    <stddev>2e-4</stddev>
-                </noise>
-                </y>
-                <z>
-                <noise type="gaussian">
-                    <mean>0.0</mean>
-                    <stddev>2e-4</stddev>
-                </noise>
-                </z>
-            </angular_velocity>
-            <linear_acceleration>
-                <x>
-                <noise type="gaussian">
-                    <mean>0.0</mean>
-                    <stddev>1.7e-2</stddev>
-                </noise>
-                </x>
-                <y>
-                <noise type="gaussian">
-                    <mean>0.0</mean>
-                    <stddev>1.7e-2</stddev>
-                </noise>
-                </y>
-                <z>
-                <noise type="gaussian">
-                    <mean>0.0</mean>
-                    <stddev>1.7e-2</stddev>
-                </noise>
-                </z>
-            </linear_acceleration>
-            </imu>
-            <plugin name="bytes_imu" filename="libgazebo_ros_imu_sensor.so">
-                <ros>
-                    <remapping>~/out:=imu</remapping>
-                </ros>
-                <initial_orientation_as_reference>false</initial_orientation_as_reference>
-            </plugin>
-        </sensor>
-    </gazebo>
-</robot>
+/home/samue/GitHub/ESDA/build/esda_sim/description/sensors/piksi.xacro

File: install/esda_sim/share/esda_sim/description/steering_wheels.xacro (robot description, xacro)
@@ -1,115 +1 @@
-<?xml version="1.0"?>
-<robot xmlns:xacro="http://www.ros.org/wiki/xacro">
-    <!-- STEERING WHEELS
-         Define the 2 front steering wheels that will turn the ESDA.
-    -->
-    <xacro:property name="steer_wheel_x_off" value="0.235"/>
-    <xacro:property name="steer_wheel_y_off" value="0.52297"/>
-    <xacro:property name="steer_wheel_z_off" value="0.208"/>
-    <!-- Define the wheels that spin -->
-    <link name="right_steering_wheel">
-        <visual>
-            <geometry>
-                <cylinder radius="${wheel_rad}" length="${wheel_len}"/>
-            </geometry>
-            <material name="light_grey"/>
-        </visual>
-        <collision>
-            <geometry>
-                <cylinder radius="${wheel_rad}" length="${wheel_len}"/>
-            </geometry>
-            <material name="light_grey"/>
-        </collision>
-        <xacro:inertial_cylinder mass="${wheel_mass}" length="${wheel_len}" radius="${wheel_rad}">
-            <origin xyz="0 0 0" rpy="0 0 0"/>
-        </xacro:inertial_cylinder>
-    </link>
-    <link name="left_steering_wheel">
-        <visual>
-            <geometry>
-                <cylinder radius="${wheel_rad}" length="${wheel_len}"/>
-            </geometry>
-            <material name="light_grey"/>
-        </visual>
-        <collision>
-            <geometry>
-                <cylinder radius="${wheel_rad}" length="${wheel_len}"/>
-            </geometry>
-            <material name="light_grey"/>
-        </collision>
-        <xacro:inertial_cylinder mass="${wheel_mass}" length="${wheel_len}" radius="${wheel_rad}">
-            <origin xyz="0 0 0" rpy="0 0 0"/>
-        </xacro:inertial_cylinder>
-    </link>
-    <!-- Define the component that will turn around z-axis which the wheels will attach to -->
-    <link name="right_steering_link">
-        <visual>
-            <geometry>
-                <cylinder radius="${wheel_rad}" length="${wheel_len}"/>
-            </geometry>
-            <material name="light_grey"/>
-        </visual>
-        <collision>
-            <geometry>
-                <cylinder radius="${wheel_rad}" length="${wheel_len}"/>
-            </geometry>
-            <material name="light_grey"/>
-        </collision>
-        <xacro:inertial_cylinder mass="${wheel_mass}" length="${wheel_len}" radius="${wheel_rad}">
-            <origin xyz="0 0 0" rpy="0 0 0"/>
-        </xacro:inertial_cylinder>
-    </link>
-    <link name="left_steering_link">
-        <visual>
-            <geometry>
-                <cylinder radius="${wheel_rad}" length="${wheel_len}"/>
-            </geometry>
-            <material name="light_grey"/>
-        </visual>
-        <collision>
-            <geometry>
-                <cylinder radius="${wheel_rad}" length="${wheel_len}"/>
-            </geometry>
-            <material name="light_grey"/>
-        </collision>
-        <xacro:inertial_cylinder mass="${wheel_mass}" length="${wheel_len}" radius="${wheel_rad}">
-            <origin xyz="0 0 0" rpy="0 0 0"/>
-        </xacro:inertial_cylinder>
-    </link>
-    <!-- Note that in the following joint definitions, when defining the
-         axis of rotation, it refers to the links axis, not base_link as
-         the wheels have been rotated 90deg for correct positioning.
-         The comments below however, are in reference to the base_link axis.
-         THe approach taken was sources from https://robotics.stackexchange.com/a/106022
-    -->
-    <!-- The steer_link will rotate around z-axis and because the wheels are jointed to this, their
-         position is relative to this and thus will follow the turn of the steer_link.
-    -->
-    <joint name="right_steer_joint" type="revolute">
-        <parent link="base_link"/>
-        <child link="right_steering_link"/>
-        <origin xyz="${steer_wheel_x_off} -${steer_wheel_y_off} -${steer_wheel_z_off}" rpy="${pi/2} 0 0 "/>
-        <axis xyz="0 -1 0"/>
-        <limit effort="100" lower="-0.41" upper="0.41" velocity="1"/>
-    </joint>
-    <joint name="left_steer_joint" type="revolute">
-        <parent link="base_link"/>
-        <child link="left_steering_link"/>
-        <origin xyz="${steer_wheel_x_off} ${steer_wheel_y_off} -${steer_wheel_z_off}" rpy="-${pi/2} 0 0 "/>
-        <axis xyz="0 1 0"/>
-        <limit effort="100" lower="-0.41" upper="0.41" velocity="1"/>
-    </joint>
-    <!-- Define the wheels rotation around the x axis so they can roll forward -->
-    <joint name="right_wheel_axle_joint" type="continuous">
-        <parent link="right_steering_link"/>
-        <child link="right_steering_wheel"/>
-        <origin xyz="0 0 0" rpy="0 0 0"/>
-        <axis xyz="0 0 -1"/>
-    </joint>
-    <joint name="left_wheel_axle_joint" type="continuous">
-        <parent link="left_steering_link"/>
-        <child link="left_steering_wheel"/>
-        <origin xyz="0 0 0" rpy="0 0 0 "/>
-        <axis xyz="0 0 1"/>
-    </joint>
-</robot>
+/home/samue/GitHub/ESDA/build/esda_sim/description/steering_wheels.xacro

File: install/esda_sim/share/esda_sim/description/util/inertial_macros.xacro (robot description, xacro)
@@ -1,32 +1 @@
-<?xml version="1.0"?>
-<robot xmlns:xacro="http://www.ros.org/wiki/xacro" >
-    <!-- Specify some standard inertial calculations https://en.wikipedia.org/wiki/List_of_moments_of_inertia -->
-    <!-- These make use of xacro's mathematical functionality -->
-    <xacro:macro name="inertial_sphere" params="mass radius *origin">
-        <inertial>
-            <xacro:insert_block name="origin"/>
-            <mass value="${mass}" />
-            <inertia ixx="${(2/5) * mass * (radius*radius)}" ixy="0.0" ixz="0.0"
-                    iyy="${(2/5) * mass * (radius*radius)}" iyz="0.0"
-                    izz="${(2/5) * mass * (radius*radius)}" />
-        </inertial>
-    </xacro:macro>
-    <xacro:macro name="inertial_box" params="mass x y z *origin">
-        <inertial>
-            <xacro:insert_block name="origin"/>
-            <mass value="${mass}" />
-            <inertia ixx="${(1/12) * mass * (y*y+z*z)}" ixy="0.0" ixz="0.0"
-                    iyy="${(1/12) * mass * (x*x+z*z)}" iyz="0.0"
-                    izz="${(1/12) * mass * (x*x+y*y)}" />
-        </inertial>
-    </xacro:macro>
-    <xacro:macro name="inertial_cylinder" params="mass length radius *origin">
-        <inertial>
-            <xacro:insert_block name="origin"/>
-            <mass value="${mass}" />
-            <inertia ixx="${(1/12) * mass * (3*radius*radius + length*length)}" ixy="0.0" ixz="0.0"
-                    iyy="${(1/12) * mass * (3*radius*radius + length*length)}" iyz="0.0"
-                    izz="${(1/2) * mass * (radius*radius)}" />
-        </inertial>
-    </xacro:macro>
-</robot>
+/home/samue/GitHub/ESDA/build/esda_sim/description/util/inertial_macros.xacro

File: install/esda_sim/share/esda_sim/description/util/materials.xacro (robot description, xacro)
@@ -1,19 +1 @@
-<?xml version="1.0"?>
-<robot xmlns:xacro="http://www.ros.org/wiki/xacro">
-    <!-- RANDOM COLOURS FOR DEBUG PURPOSES -->
-    <material name="white">
-        <color rgba="1 1 1 0.3"/>
-    </material>
-    <material name="light_grey">
-        <color rgba="0.9 0.9 0.9 0.4"/>
-    </material>
-    <material name="black">
-        <color rgba="0.2 0.2 0.2 0.4"/>
-    </material>
-    <material name="blue">
-        <color rgba="0.2 0.2 1 1"/>
-    </material>
-    <material name="orange">
-        <color rgba="1 0.3 0.1 1"/>
-    </material>
-</robot>
+/home/samue/GitHub/ESDA/build/esda_sim/description/util/materials.xacro

File: install/esda_sim/share/esda_sim/description/wheels.xacro (robot description, xacro)
@@ -1,26 +1 @@
-<?xml version="1.0"?>
-<robot xmlns:xacro="http://www.ros.org/wiki/xacro">
-    <!-- WHEEL LINKS
-         these define the 4 wheels and their attachment to
-         the vehicle. Note due to complexity of CAD, wheels are
-         parallel and upright as they don't need accurate modelling
-    -->
-    <xacro:property name="wheel_rad" value="0.1325"/>
-    <xacro:property name="wheel_len" value="0.07"/>
-    <xacro:property name="wheel_mass" value="2"/>
-    <xacro:include filename="drive_wheels.xacro"/>
-    <xacro:include filename="caster_wheels.xacro"/>
-    <!-- Adding colours to wheels for gazebo -->
-    <gazebo reference="left_drive_wheel">
-        <material>Gazebo/Black</material>
-    </gazebo>
-    <gazebo reference="right_drive_wheel">
-        <material>Gazebo/Black</material>
-    </gazebo>
-    <gazebo reference="left_caster_wheel">
-        <material>Gazebo/Black</material>
-    </gazebo>
-    <gazebo reference="right_caster_wheel">
-        <material>Gazebo/Black</material>
-    </gazebo>
-</robot>
+/home/samue/GitHub/ESDA/build/esda_sim/description/wheels.xacro
